File: schema/valve/usb.sch (KiCad schematic (older format))
At the start: 11 parts, among them J1 USB_2_VALID, Q28 bc857, Q29 bc847

Commit message: Schema, svg and png.
Parts:
- renumbered Q28 to Q32, Q29 to Q33, R84 to R101, R86 to R102, R81 to R103, R87 to R104, R82 to R105, R85 to R106, R83 to R107
Changed lines of the file:
@@
-EESchema Schematic File Version 2  date Tue 03 Apr 2012 09:00:56 PM MSK
+EESchema Schematic File Version 2  date Wed 04 Apr 2012 04:27:02 PM MSK
 LIBS:power
 LIBS:device
@@
 $Descr A4 11700 8267
 encoding utf-8
-Sheet 4 28
+Sheet 25 27
 Title ""
-Date "3 apr 2012"
+Date "4 apr 2012"
 Rev ""
 Comp ""
@@
 en
 $Comp
-L GND #PWR62
+L GND #PWR091
 U 1 1 4F79F38D
 P 8800 4300
-F 0 "#PWR62" H 8800 4300 30  0001 C CNN
+F 0 "#PWR091" H 8800 4300 30  0001 C CNN
 F 1 "GND" H 8800 4230 30  0001 C CNN
 	1    8800 4300
@@
 $EndComp
 $Comp
-L R R85
+L R R106
 U 1 1 4F79F383
 P 8800 3750
-F 0 "R85" V 8880 3750 50  0000 C CNN
+F 0 "R106" V 8880 3750 50  0000 C CNN
 F 1 "10k" V 8800 3750 50  0000 C CNN
 	1    8800 3750
@@
 $EndComp
 $Comp
-L R R83
+L R R107
 U 1 1 4F79F376
 P 9350 3200
-F 0 "R83" V 9430 3200 50  0000 C CNN
+F 0 "R107" V 9430 3200 50  0000 C CNN
 F 1 "1k" V 9350 3200 50  0000 C CNN
 	1    9350 3200
@@
 $EndComp
 $Comp
-L GND #PWR61
+L GND #PWR092
 U 1 1 4F79F36D
 P 8200 3800
-F 0 "#PWR61" H 8200 3800 30  0001 C CNN
+F 0 "#PWR092" H 8200 3800 30  0001 C CNN
 F 1 "GND" H 8200 3730 30  0001 C CNN
 	1    8200 3800
@@
 $EndComp
 $Comp
-L NPN Q29
+L NPN Q33
 U 1 1 4F79F34C
 P 8300 3200
-F 0 "Q29" H 8300 3050 50  0000 R CNN
+F 0 "Q33" H 8300 3050 50  0000 R CNN
 F 1 "bc847" H 8300 3350 50  0000 R CNN
 	1    8300 3200
@@
 $EndComp
 $Comp
-L R R82
+L R R105
 U 1 1 4F79F31F
 P 6850 2800
-F 0 "R82" V 6930 2800 50  0000 C CNN
+F 0 "R105" V 6930 2800 50  0000 C CNN
 F 1 "1k" V 6850 2800 50  0000 C CNN
 	1    6850 2800
@@
 usb-vcc
 $Comp
-L R R81
+L R R103
 U 1 1 4F79F29C
 P 6300 2250
-F 0 "R81" V 6380 2250 50  0000 C CNN
+F 0 "R103" V 6380 2250 50  0000 C CNN
 F 1 "10k" V 6300 2250 50  0000 C CNN
 	1    6300 2250
@@
 $EndComp
 $Comp
-L PNP Q28
+L PNP Q32
 U 1 1 4F79F27D
 P 5800 2800
-F 0 "Q28" H 5800 2650 60  0000 R CNN
+F 0 "Q32" H 5800 2650 60  0000 R CNN
 F 1 "bc857" H 5800 2950 60  0000 R CNN
 	1    5800 2800
@@
 d-
 $Comp
-L GND #PWR60
+L GND #PWR093
 U 1 1 4F79EA74
 P 5200 3750
-F 0 "#PWR60" H 5200 3750 30  0001 C CNN
+F 0 "#PWR093" H 5200 3750 30  0001 C CNN
 F 1 "GND" H 5200 3680 30  0001 C CNN
 	1    5200 3750
@@
 usb-vcc
 $Comp
-L GND #PWR63
+L GND #PWR094
 U 1 1 4F79EA26
 P 5500 4600
-F 0 "#PWR63" H 5500 4600 30  0001 C CNN
+F 0 "#PWR094" H 5500 4600 30  0001 C CNN
 F 1 "GND" H 5500 4530 30  0001 C CNN
 	1    5500 4600
@@
 $EndComp
 $Comp
-L R R84
+L R R101
 U 1 1 4F79E9FF
 P 5700 3550
-F 0 "R84" V 5780 3550 50  0000 C CNN
+F 0 "R101" V 5780 3550 50  0000 C CNN
 F 1 "1k5" V 5700 3550 50  0000 C CNN
 	1    5700 3550
@@
 $EndComp
 $Comp
-L R R87
+L R R104
 U 1 1 4F79E9AD
 P 6700 4200
-F 0 "R87" V 6780 4200 50  0000 C CNN
+F 0 "R104" V 6780 4200 50  0000 C CNN
 F 1 "22" V 6700 4200 50  0000 C CNN
 	1    6700 4200
@@
 $EndComp
 $Comp
-L R R86
+L R R102
 U 1 1 4F79E9A1
 P 6100 4100
-F 0 "R86" V 6180 4100 50  0000 C CNN
+F 0 "R102" V 6180 4100 50  0000 C CNN
 F 1 "22" V 6100 4100 50  0000 C CNN
 	1    6100 4100
