File: schema/valve-hm/output2.sch (KiCad schematic (older format))
At the start: 7 parts, among them Q4 MOSFET_N, Q5 MOSFET_N, U4 MC34152

Commit message: Разводка платы.
Parts:
- D3, D4: value DIODE -> 1N4148
Changed lines of the file:
@@
-EESchema Schematic File Version 2  date 15/06/2012 18:13:53
+EESchema Schematic File Version 2  date Sat 16 Jun 2012 11:54:35 AM MSK
 LIBS:power
 LIBS:device
@@
 Sheet 6 7
 Title ""
-Date "15 jun 2012"
+Date "16 jun 2012"
 Rev ""
 Comp ""
@@
 AR Path="/4FDB33F6/4FDB2ED0" Ref="R37"  Part="1"
 AR Path="/4FDB2BC5/4FDB2ED0" Ref="R39"  Part="1"
-F 0 "R37" V 9230 2100 50  0000 C CNN
+F 0 "R39" V 9230 2100 50  0000 C CNN
 F 1 "10" V 9150 2100 50  0000 C CNN
 	1    9150 2100
@@
 AR Path="/4FDB33F6/4FDB2ECF" Ref="Q5"  Part="1"
 AR Path="/4FDB2BC5/4FDB2ECF" Ref="Q7"  Part="1"
-F 0 "Q5" H 9810 2270 60  0000 R CNN
+F 0 "Q7" H 9810 2270 60  0000 R CNN
 F 1 "MOSFET_N" H 9810 1950 60  0000 R CNN
 	1    9800 2100
@@
 AR Path="/4FDB33F6/4FDB2ECD" Ref="D4"  Part="1"
 AR Path="/4FDB2BC5/4FDB2ECD" Ref="D6"  Part="1"
-F 0 "D4" H 9900 1600 40  0000 C CNN
-F 1 "DIODE" H 9900 1400 40  0000 C CNN
+F 0 "D6" H 9900 1600 40  0000 C CNN
+F 1 "1N4148" H 9900 1400 40  0000 C CNN
 	1    9900 1500
 	0    -1   -1   0
@@
 AR Path="/4FDB33F6/4FDB2DC3" Ref="D3"  Part="1"
 AR Path="/4FDB2BC5/4FDB2DC3" Ref="D5"  Part="1"
-F 0 "D3" H 7400 1600 40  0000 C CNN
-F 1 "DIODE" H 7400 1400 40  0000 C CNN
+F 0 "D5" H 7400 1600 40  0000 C CNN
+F 1 "1N4148" H 7400 1400 40  0000 C CNN
 	1    7400 1500
 	0    -1   -1   0
@@
 AR Path="/4FDB33F6/4FDB2C4B" Ref="Q4"  Part="1"
 AR Path="/4FDB2BC5/4FDB2C4B" Ref="Q6"  Part="1"
-F 0 "Q4" H 7310 2270 60  0000 R CNN
+F 0 "Q6" H 7310 2270 60  0000 R CNN
 F 1 "MOSFET_N" H 7310 1950 60  0000 R CNN
 	1    7300 2100
@@
 AR Path="/4FDB33F6/4FDB2C18" Ref="R36"  Part="1"
 AR Path="/4FDB2BC5/4FDB2C18" Ref="R38"  Part="1"
-F 0 "R36" V 6730 2100 50  0000 C CNN
+F 0 "R38" V 6730 2100 50  0000 C CNN
 F 1 "10" V 6650 2100 50  0000 C CNN
 	1    6650 2100
@@
 AR Path="/4FDB33F6/4FDB2BFB" Ref="U4"  Part="1"
 AR Path="/4FDB2BC5/4FDB2BFB" Ref="U5"  Part="1"
-F 0 "U4" H 5800 4100 60  0000 C CNN
+F 0 "U5" H 5800 4100 60  0000 C CNN
 F 1 "MC34152" H 5800 3750 60  0000 C CNN
 	1    5800 3750
