File: schema/valve-hm/valve-hm.sch (KiCad schematic (older format))
At the start: 67 parts, among them K1 swd, P1 24v, P10 port-out, P11 port-out, P12 port-out, P13 port-out, P14 port-out, P15 port-out, P16 port-out, P2 op-mode, P3 3.3v, P4 10v, P5 flash-mode, P6 3.3v, P7 10v, P8 i2c, P9 port-out, U1 MINI-USB-B, U2 NCP3063, U3 NCP3063, X1 8MHz

Commit message: Valve-hm is ready. It's digital IO board which can control up to 20 io pins. It is rquipt with 3 LEDs, 2 operating mode switches, USB port and TWI interface.
Parts:
- removed C10, C9: 1m, symbol C
- removed C13, C3, C4, C7, C8: 100n, symbol C
- removed C15: 1u, symbol C
- removed C2: 4u7, symbol C
- removed C5, C6: 2.2n, symbol C
- removed D1, D2: 1N5819, symbol DIODESCH
- removed L1, L2: INDUCTOR, symbol INDUCTOR
- removed P1: 24v, symbol CONN_4
- removed P10, P11, P12, P13, P14, P15, P16, P9: port-out, symbol CONN_2
- removed P4, P7: 10v, symbol CONN_2
- removed P6: 3.3v, symbol CONN_2
- removed R10: 50k, symbol R
- removed R4, R5, R6: 1R5, symbol R
- removed R7: 12k, symbol R
- removed R8: 10k, symbol R
- removed R9: 20k, symbol R
- removed U2, U3: NCP3063, symbol NCP3063
- added D1, D2, D3: LED, symbol LED
- added P1: CONN_12, symbol CONN_12
- added P4: CONN_8, symbol CONN_8
- R1, R2, R3: value 1R5 -> 500
- R20: value 360 -> 50
Connections:
- net labels added: io1, io10, io11, io12, io13, io14, io15, io16, io17, io18, io19, io2, io20, io3, io4, io5, io6, io7, io8, io9, led1, led2, led3
- net labels removed: 10v, 10v-out, 24v, buck-out, in3, in4, out-int1, out-int2, out-int3, out-int4, out1, out2, out3, out4, pa10, pa15, pa4, pa5, pa6, pa7, pa8, pa9, pb0, pb1, pb12, pb13, pb14, pb15, pb2, pb3, pb4
- wire segments 260 -> 152
- no-connect marks 18 -> 3
Other:
- moved on the sheet: P2, P5, R11, R12, R13, R14, R15, R16, U1
