File: schema/valve-power/input.sch (KiCad schematic (older format))
At the start: 5 parts, among them Q1 bc847

Commit message: Valve-power board is in progress.
Parts:
- renumbered R24 to R11, R25 to R12, R26 to R13, R27 to R14
Changed lines of the file:
@@
-EESchema Schematic File Version 2  date Sat 16 Jun 2012 04:56:37 PM MSK
+EESchema Schematic File Version 2  date Sat 16 Jun 2012 11:30:21 PM MSK
 LIBS:power
 LIBS:device
@@
 $Descr A4 11700 8267
 encoding utf-8
-Sheet 7 17
+Sheet 4 17
 Title ""
 Date "16 jun 2012"
@@
 $EndDescr
 $Comp
-L VDD #PWR049
+L VDD #PWR030
 U 1 1 4FDB399C
 P 5800 2050
-AR Path="/4FDB3936/4FDB399C" Ref="#PWR049"  Part="1"
-AR Path="/4FDB3935/4FDB399C" Ref="#PWR052"  Part="1"
-AR Path="/4FDB3921/4FDB399C" Ref="#PWR055"  Part="1"
-AR Path="/4FDB299D/4FDB399C" Ref="#PWR068"  Part="1"
-F 0 "#PWR068" H 5800 2150 30  0001 C CNN
+AR Path="/4FDC7DE6/4FDB399C" Ref="#PWR030"  Part="1"
+AR Path="/4FDC7DE5/4FDB399C" Ref="#PWR033"  Part="1"
+AR Path="/4FDC7DE4/4FDB399C" Ref="#PWR036"  Part="1"
+AR Path="/4FDC7DE3/4FDB399C" Ref="#PWR039"  Part="1"
+AR Path="/4FDC7DB7/4FDB399C" Ref="#PWR042"  Part="1"
+AR Path="/4FDC7DB6/4FDB399C" Ref="#PWR045"  Part="1"
+AR Path="/4FDC7DB5/4FDB399C" Ref="#PWR048"  Part="1"
+AR Path="/4FDC7DB4/4FDB399C" Ref="#PWR051"  Part="1"
+AR Path="/4FDB299D/4FDB399C" Ref="#PWR069"  Part="1"
+AR Path="/4FDB3921/4FDB399C" Ref="#PWR072"  Part="1"
+AR Path="/4FDB3935/4FDB399C" Ref="#PWR075"  Part="1"
+AR Path="/4FDB3936/4FDB399C" Ref="#PWR078"  Part="1"
+F 0 "#PWR078" H 5800 2150 30  0001 C CNN
 F 1 "VDD" H 5800 2160 30  0000 C CNN
 	1    5800 2050
@@
 	6750 3250 7150 3250
 $Comp
-L R R26
+L R R13
 U 1 1 4FDB2AE7
 P 5800 2550
-AR Path="/4FDB3936/4FDB2AE7" Ref="R26"  Part="1"
-AR Path="/4FDB3935/4FDB2AE7" Ref="R30"  Part="1"
-AR Path="/4FDB3921/4FDB2AE7" Ref="R34"  Part="1"
-AR Path="/4FDB299D/4FDB2AE7" Ref="R42"  Part="1"
-F 0 "R42" V 5880 2550 50  0000 C CNN
+AR Path="/4FDC7DE6/4FDB2AE7" Ref="R13"  Part="1"
+AR Path="/4FDC7DE5/4FDB2AE7" Ref="R17"  Part="1"
+AR Path="/4FDC7DE4/4FDB2AE7" Ref="R21"  Part="1"
+AR Path="/4FDC7DE3/4FDB2AE7" Ref="R25"  Part="1"
+AR Path="/4FDC7DB7/4FDB2AE7" Ref="R29"  Part="1"
+AR Path="/4FDC7DB6/4FDB2AE7" Ref="R33"  Part="1"
+AR Path="/4FDC7DB5/4FDB2AE7" Ref="R37"  Part="1"
+AR Path="/4FDC7DB4/4FDB2AE7" Ref="R41"  Part="1"
+AR Path="/4FDB299D/4FDB2AE7" Ref="R61"  Part="1"
+AR Path="/4FDB3921/4FDB2AE7" Ref="R65"  Part="1"
+AR Path="/4FDB3935/4FDB2AE7" Ref="R69"  Part="1"
+AR Path="/4FDB3936/4FDB2AE7" Ref="R73"  Part="1"
+F 0 "R13" V 5880 2550 50  0000 C CNN
 F 1 "33k" V 5800 2550 50  0000 C CNN
 	1    5800 2550
@@
 out
 $Comp
-L R R27
+L R R14
 U 1 1 4FDB2AA4
 P 6500 3250
-AR Path="/4FDB3936/4FDB2AA4" Ref="R27"  Part="1"
-AR Path="/4FDB3935/4FDB2AA4" Ref="R31"  Part="1"
-AR Path="/4FDB3921/4FDB2AA4" Ref="R35"  Part="1"
-AR Path="/4FDB299D/4FDB2AA4" Ref="R43"  Part="1"
-F 0 "R43" V 6580 3250 50  0000 C CNN
+AR Path="/4FDC7DE6/4FDB2AA4" Ref="R14"  Part="1"
+AR Path="/4FDC7DE5/4FDB2AA4" Ref="R18"  Part="1"
+AR Path="/4FDC7DE4/4FDB2AA4" Ref="R22"  Part="1"
+AR Path="/4FDC7DE3/4FDB2AA4" Ref="R26"  Part="1"
+AR Path="/4FDC7DB7/4FDB2AA4" Ref="R30"  Part="1"
+AR Path="/4FDC7DB6/4FDB2AA4" Ref="R34"  Part="1"
+AR Path="/4FDC7DB5/4FDB2AA4" Ref="R38"  Part="1"
+AR Path="/4FDC7DB4/4FDB2AA4" Ref="R42"  Part="1"
+AR Path="/4FDB299D/4FDB2AA4" Ref="R62"  Part="1"
+AR Path="/4FDB3921/4FDB2AA4" Ref="R66"  Part="1"
+AR Path="/4FDB3935/4FDB2AA4" Ref="R70"  Part="1"
+AR Path="/4FDB3936/4FDB2AA4" Ref="R74"  Part="1"
+F 0 "R14" V 6580 3250 50  0000 C CNN
 F 1 "2k4" V 6500 3250 50  0000 C CNN
 	1    6500 3250
@@
 $EndComp
 $Comp
-L GND #PWR050
+L GND #PWR031
 U 1 1 4FDB2A6B
 P 4600 4700
-AR Path="/4FDB3936/4FDB2A6B" Ref="#PWR050"  Part="1"
-AR Path="/4FDB3935/4FDB2A6B" Ref="#PWR053"  Part="1"
-AR Path="/4FDB3921/4FDB2A6B" Ref="#PWR056"  Part="1"
-AR Path="/4FDB299D/4FDB2A6B" Ref="#PWR069"  Part="1"
-F 0 "#PWR069" H 4600 4700 30  0001 C CNN
+AR Path="/4FDC7DE6/4FDB2A6B" Ref="#PWR031"  Part="1"
+AR Path="/4FDC7DE5/4FDB2A6B" Ref="#PWR034"  Part="1"
+AR Path="/4FDC7DE4/4FDB2A6B" Ref="#PWR037"  Part="1"
+AR Path="/4FDC7DE3/4FDB2A6B" Ref="#PWR040"  Part="1"
+AR Path="/4FDC7DB7/4FDB2A6B" Ref="#PWR043"  Part="1"
+AR Path="/4FDC7DB6/4FDB2A6B" Ref="#PWR046"  Part="1"
+AR Path="/4FDC7DB5/4FDB2A6B" Ref="#PWR049"  Part="1"
+AR Path="/4FDC7DB4/4FDB2A6B" Ref="#PWR052"  Part="1"
+AR Path="/4FDB299D/4FDB2A6B" Ref="#PWR070"  Part="1"
+AR Path="/4FDB3921/4FDB2A6B" Ref="#PWR073"  Part="1"
+AR Path="/4FDB3935/4FDB2A6B" Ref="#PWR076"  Part="1"
+AR Path="/4FDB3936/4FDB2A6B" Ref="#PWR079"  Part="1"
+F 0 "#PWR079" H 4600 4700 30  0001 C CNN
 F 1 "GND" H 4600 4630 30  0001 C CNN
 	1    4600 4700
@@
 $EndComp
 $Comp
-L GND #PWR051
+L GND #PWR032
 U 1 1 4FDB2A62
 P 5800 4550
-AR Path="/4FDB3936/4FDB2A62" Ref="#PWR051"  Part="1"
-AR Path="/4FDB3935/4FDB2A62" Ref="#PWR054"  Part="1"
-AR Path="/4FDB3921/4FDB2A62" Ref="#PWR057"  Part="1"
-AR Path="/4FDB299D/4FDB2A62" Ref="#PWR070"  Part="1"
-F 0 "#PWR070" H 5800 4550 30  0001 C CNN
+AR Path="/4FDC7DE6/4FDB2A62" Ref="#PWR032"  Part="1"
+AR Path="/4FDC7DE5/4FDB2A62" Ref="#PWR035"  Part="1"
+AR Path="/4FDC7DE4/4FDB2A62" Ref="#PWR038"  Part="1"
+AR Path="/4FDC7DE3/4FDB2A62" Ref="#PWR041"  Part="1"
+AR Path="/4FDC7DB7/4FDB2A62" Ref="#PWR044"  Part="1"
+AR Path="/4FDC7DB6/4FDB2A62" Ref="#PWR047"  Part="1"
+AR Path="/4FDC7DB5/4FDB2A62" Ref="#PWR050"  Part="1"
+AR Path="/4FDC7DB4/4FDB2A62" Ref="#PWR053"  Part="1"
+AR Path="/4FDB299D/4FDB2A62" Ref="#PWR071"  Part="1"
+AR Path="/4FDB3921/4FDB2A62" Ref="#PWR074"  Part="1"
+AR Path="/4FDB3935/4FDB2A62" Ref="#PWR077"  Part="1"
+AR Path="/4FDB3936/4FDB2A62" Ref="#PWR080"  Part="1"
+F 0 "#PWR080" H 5800 4550 30  0001 C CNN
 F 1 "GND" H 5800 4480 30  0001 C CNN
 	1    5800 4550
@@
 in-24v
 $Comp
-L R R25
+L R R12
 U 1 1 4FDB29FE
 P 5050 3600
-AR Path="/4FDB3936/4FDB29FE" Ref="R25"  Part="1"
-AR Path="/4FDB3935/4FDB29FE" Ref="R29"  Part="1"
-AR Path="/4FDB3921/4FDB29FE" Ref="R33"  Part="1"
-AR Path="/4FDB299D/4FDB29FE" Ref="R41"  Part="1"
-F 0 "R41" V 5130 3600 50  0000 C CNN
+AR Path="/4FDC7DE6/4FDB29FE" Ref="R12"  Part="1"
+AR Path="/4FDC7DE5/4FDB29FE" Ref="R16"  Part="1"
+AR Path="/4FDC7DE4/4FDB29FE" Ref="R20"  Part="1"
+AR Path="/4FDC7DE3/4FDB29FE" Ref="R24"  Part="1"
+AR Path="/4FDC7DB7/4FDB29FE" Ref="R28"  Part="1"
+AR Path="/4FDC7DB6/4FDB29FE" Ref="R32"  Part="1"
+AR Path="/4FDC7DB5/4FDB29FE" Ref="R36"  Part="1"
+AR Path="/4FDC7DB4/4FDB29FE" Ref="R40"  Part="1"
+AR Path="/4FDB299D/4FDB29FE" Ref="R60"  Part="1"
+AR Path="/4FDB3921/4FDB29FE" Ref="R64"  Part="1"
+AR Path="/4FDB3935/4FDB29FE" Ref="R68"  Part="1"
+AR Path="/4FDB3936/4FDB29FE" Ref="R72"  Part="1"
+F 0 "R12" V 5130 3600 50  0000 C CNN
 F 1 "2k4" V 5050 3600 50  0000 C CNN
 	1    5050 3600
@@
 $EndComp
 $Comp
-L R R24
+L R R11
 U 1 1 4FDB29E5
 P 4600 4250
-AR Path="/4FDB3936/4FDB29E5" Ref="R24"  Part="1"
-AR Path="/4FDB3935/4FDB29E5" Ref="R28"  Part="1"
-AR Path="/4FDB3921/4FDB29E5" Ref="R32"  Part="1"
-AR Path="/4FDB299D/4FDB29E5" Ref="R40"  Part="1"
-F 0 "R40" V 4680 4250 50  0000 C CNN
+AR Path="/4FDC7DE6/4FDB29E5" Ref="R11"  Part="1"
+AR Path="/4FDC7DE5/4FDB29E5" Ref="R15"  Part="1"
+AR Path="/4FDC7DE4/4FDB29E5" Ref="R19"  Part="1"
+AR Path="/4FDC7DE3/4FDB29E5" Ref="R23"  Part="1"
+AR Path="/4FDC7DB7/4FDB29E5" Ref="R27"  Part="1"
+AR Path="/4FDC7DB6/4FDB29E5" Ref="R31"  Part="1"
+AR Path="/4FDC7DB5/4FDB29E5" Ref="R35"  Part="1"
+AR Path="/4FDC7DB4/4FDB29E5" Ref="R39"  Part="1"
+AR Path="/4FDB299D/4FDB29E5" Ref="R59"  Part="1"
+AR Path="/4FDB3921/4FDB29E5" Ref="R63"  Part="1"
+AR Path="/4FDB3935/4FDB29E5" Ref="R67"  Part="1"
+AR Path="/4FDB3936/4FDB29E5" Ref="R71"  Part="1"
+F 0 "R11" V 4680 4250 50  0000 C CNN
 F 1 "33k" V 4600 4250 50  0000 C CNN
 	1    4600 4250
@@
 U 1 1 4FDB29D2
 P 5700 3600
-AR Path="/4FDB3936/4FDB29D2" Ref="Q1"  Part="1"
-AR Path="/4FDB3935/4FDB29D2" Ref="Q2"  Part="1"
-AR Path="/4FDB3921/4FDB29D2" Ref="Q3"  Part="1"
-AR Path="/4FDB299D/4FDB29D2" Ref="Q8"  Part="1"
-F 0 "Q8" H 5700 3450 50  0000 R CNN
+AR Path="/4FDC7DE6/4FDB29D2" Ref="Q1"  Part="1"
+AR Path="/4FDC7DE5/4FDB29D2" Ref="Q2"  Part="1"
+AR Path="/4FDC7DE4/4FDB29D2" Ref="Q3"  Part="1"
+AR Path="/4FDC7DE3/4FDB29D2" Ref="Q4"  Part="1"
+AR Path="/4FDC7DB7/4FDB29D2" Ref="Q5"  Part="1"
+AR Path="/4FDC7DB6/4FDB29D2" Ref="Q6"  Part="1"
+AR Path="/4FDC7DB5/4FDB29D2" Ref="Q7"  Part="1"
+AR Path="/4FDC7DB4/4FDB29D2" Ref="Q8"  Part="1"
+AR Path="/4FDB299D/4FDB29D2" Ref="Q17"  Part="1"
+AR Path="/4FDB3921/4FDB29D2" Ref="Q18"  Part="1"
+AR Path="/4FDB3935/4FDB29D2" Ref="Q19"  Part="1"
+AR Path="/4FDB3936/4FDB29D2" Ref="Q20"  Part="1"
+F 0 "Q1" H 5700 3450 50  0000 R CNN
 F 1 "bc847" H 5700 3750 50  0000 R CNN
 	1    5700 3600
