File: schema/valve-power/input.sch (KiCad schematic (older format))
At the start: 5 parts, among them Q1 bc847

Commit message: Power supply board is ready.
Changed lines of the file:
@@
-EESchema Schematic File Version 2  date Sun 17 Jun 2012 09:58:46 PM MSK
+EESchema Schematic File Version 2  date Mon 18 Jun 2012 12:08:36 AM MSK
 LIBS:power
 LIBS:device
@@
 $Descr A4 11700 8267
 encoding utf-8
-Sheet 4 17
+Sheet 5 17
 Title ""
 Date "17 jun 2012"
@@
 $EndDescr
 $Comp
-L VDD #PWR030
+L VDD #PWR031
 U 1 1 4FDB399C
 P 5800 2050
-AR Path="/4FDC7DE6/4FDB399C" Ref="#PWR030"  Part="1"
-AR Path="/4FDC7DE5/4FDB399C" Ref="#PWR033"  Part="1"
-AR Path="/4FDC7DE4/4FDB399C" Ref="#PWR036"  Part="1"
-AR Path="/4FDC7DE3/4FDB399C" Ref="#PWR039"  Part="1"
-AR Path="/4FDC7DB7/4FDB399C" Ref="#PWR042"  Part="1"
-AR Path="/4FDC7DB6/4FDB399C" Ref="#PWR045"  Part="1"
-AR Path="/4FDC7DB5/4FDB399C" Ref="#PWR048"  Part="1"
-AR Path="/4FDC7DB4/4FDB399C" Ref="#PWR051"  Part="1"
-AR Path="/4FDB299D/4FDB399C" Ref="#PWR069"  Part="1"
-AR Path="/4FDB3921/4FDB399C" Ref="#PWR072"  Part="1"
-AR Path="/4FDB3935/4FDB399C" Ref="#PWR075"  Part="1"
-AR Path="/4FDB3936/4FDB399C" Ref="#PWR078"  Part="1"
-F 0 "#PWR078" H 5800 2150 30  0001 C CNN
+AR Path="/4FDC7DE6/4FDB399C" Ref="#PWR031"  Part="1"
+AR Path="/4FDC7DE5/4FDB399C" Ref="#PWR034"  Part="1"
+AR Path="/4FDC7DE4/4FDB399C" Ref="#PWR037"  Part="1"
+AR Path="/4FDC7DE3/4FDB399C" Ref="#PWR040"  Part="1"
+AR Path="/4FDC7DB7/4FDB399C" Ref="#PWR043"  Part="1"
+AR Path="/4FDC7DB6/4FDB399C" Ref="#PWR046"  Part="1"
+AR Path="/4FDC7DB5/4FDB399C" Ref="#PWR049"  Part="1"
+AR Path="/4FDC7DB4/4FDB399C" Ref="#PWR052"  Part="1"
+AR Path="/4FDB299D/4FDB399C" Ref="#PWR073"  Part="1"
+AR Path="/4FDB3921/4FDB399C" Ref="#PWR076"  Part="1"
+AR Path="/4FDB3935/4FDB399C" Ref="#PWR079"  Part="1"
+AR Path="/4FDB3936/4FDB399C" Ref="#PWR082"  Part="1"
+F 0 "#PWR082" H 5800 2150 30  0001 C CNN
 F 1 "VDD" H 5800 2160 30  0000 C CNN
 	1    5800 2050
@@
 AR Path="/4FDB3935/4FDB2AE7" Ref="R69"  Part="1"
 AR Path="/4FDB3936/4FDB2AE7" Ref="R73"  Part="1"
-F 0 "R13" V 5880 2550 50  0000 C CNN
+F 0 "R73" V 5880 2550 50  0000 C CNN
 F 1 "33k" V 5800 2550 50  0000 C CNN
 	1    5800 2550
@@
 AR Path="/4FDB3935/4FDB2AA4" Ref="R70"  Part="1"
 AR Path="/4FDB3936/4FDB2AA4" Ref="R74"  Part="1"
-F 0 "R14" V 6580 3250 50  0000 C CNN
+F 0 "R74" V 6580 3250 50  0000 C CNN
 F 1 "2k4" V 6500 3250 50  0000 C CNN
 	1    6500 3250
@@
 $EndComp
 $Comp
-L GND #PWR031
+L GND #PWR032
 U 1 1 4FDB2A6B
 P 4600 4700
-AR Path="/4FDC7DE6/4FDB2A6B" Ref="#PWR031"  Part="1"
-AR Path="/4FDC7DE5/4FDB2A6B" Ref="#PWR034"  Part="1"
-AR Path="/4FDC7DE4/4FDB2A6B" Ref="#PWR037"  Part="1"
-AR Path="/4FDC7DE3/4FDB2A6B" Ref="#PWR040"  Part="1"
-AR Path="/4FDC7DB7/4FDB2A6B" Ref="#PWR043"  Part="1"
-AR Path="/4FDC7DB6/4FDB2A6B" Ref="#PWR046"  Part="1"
-AR Path="/4FDC7DB5/4FDB2A6B" Ref="#PWR049"  Part="1"
-AR Path="/4FDC7DB4/4FDB2A6B" Ref="#PWR052"  Part="1"
-AR Path="/4FDB299D/4FDB2A6B" Ref="#PWR070"  Part="1"
-AR Path="/4FDB3921/4FDB2A6B" Ref="#PWR073"  Part="1"
-AR Path="/4FDB3935/4FDB2A6B" Ref="#PWR076"  Part="1"
-AR Path="/4FDB3936/4FDB2A6B" Ref="#PWR079"  Part="1"
-F 0 "#PWR079" H 4600 4700 30  0001 C CNN
+AR Path="/4FDC7DE6/4FDB2A6B" Ref="#PWR032"  Part="1"
+AR Path="/4FDC7DE5/4FDB2A6B" Ref="#PWR035"  Part="1"
+AR Path="/4FDC7DE4/4FDB2A6B" Ref="#PWR038"  Part="1"
+AR Path="/4FDC7DE3/4FDB2A6B" Ref="#PWR041"  Part="1"
+AR Path="/4FDC7DB7/4FDB2A6B" Ref="#PWR044"  Part="1"
+AR Path="/4FDC7DB6/4FDB2A6B" Ref="#PWR047"  Part="1"
+AR Path="/4FDC7DB5/4FDB2A6B" Ref="#PWR050"  Part="1"
+AR Path="/4FDC7DB4/4FDB2A6B" Ref="#PWR053"  Part="1"
+AR Path="/4FDB299D/4FDB2A6B" Ref="#PWR074"  Part="1"
+AR Path="/4FDB3921/4FDB2A6B" Ref="#PWR077"  Part="1"
+AR Path="/4FDB3935/4FDB2A6B" Ref="#PWR080"  Part="1"
+AR Path="/4FDB3936/4FDB2A6B" Ref="#PWR083"  Part="1"
+F 0 "#PWR083" H 4600 4700 30  0001 C CNN
 F 1 "GND" H 4600 4630 30  0001 C CNN
 	1    4600 4700
@@
 $EndComp
 $Comp
-L GND #PWR032
+L GND #PWR033
 U 1 1 4FDB2A62
 P 5800 4550
-AR Path="/4FDC7DE6/4FDB2A62" Ref="#PWR032"  Part="1"
-AR Path="/4FDC7DE5/4FDB2A62" Ref="#PWR035"  Part="1"
-AR Path="/4FDC7DE4/4FDB2A62" Ref="#PWR038"  Part="1"
-AR Path="/4FDC7DE3/4FDB2A62" Ref="#PWR041"  Part="1"
-AR Path="/4FDC7DB7/4FDB2A62" Ref="#PWR044"  Part="1"
-AR Path="/4FDC7DB6/4FDB2A62" Ref="#PWR047"  Part="1"
-AR Path="/4FDC7DB5/4FDB2A62" Ref="#PWR050"  Part="1"
-AR Path="/4FDC7DB4/4FDB2A62" Ref="#PWR053"  Part="1"
-AR Path="/4FDB299D/4FDB2A62" Ref="#PWR071"  Part="1"
-AR Path="/4FDB3921/4FDB2A62" Ref="#PWR074"  Part="1"
-AR Path="/4FDB3935/4FDB2A62" Ref="#PWR077"  Part="1"
-AR Path="/4FDB3936/4FDB2A62" Ref="#PWR080"  Part="1"
-F 0 "#PWR080" H 5800 4550 30  0001 C CNN
+AR Path="/4FDC7DE6/4FDB2A62" Ref="#PWR033"  Part="1"
+AR Path="/4FDC7DE5/4FDB2A62" Ref="#PWR036"  Part="1"
+AR Path="/4FDC7DE4/4FDB2A62" Ref="#PWR039"  Part="1"
+AR Path="/4FDC7DE3/4FDB2A62" Ref="#PWR042"  Part="1"
+AR Path="/4FDC7DB7/4FDB2A62" Ref="#PWR045"  Part="1"
+AR Path="/4FDC7DB6/4FDB2A62" Ref="#PWR048"  Part="1"
+AR Path="/4FDC7DB5/4FDB2A62" Ref="#PWR051"  Part="1"
+AR Path="/4FDC7DB4/4FDB2A62" Ref="#PWR054"  Part="1"
+AR Path="/4FDB299D/4FDB2A62" Ref="#PWR075"  Part="1"
+AR Path="/4FDB3921/4FDB2A62" Ref="#PWR078"  Part="1"
+AR Path="/4FDB3935/4FDB2A62" Ref="#PWR081"  Part="1"
+AR Path="/4FDB3936/4FDB2A62" Ref="#PWR084"  Part="1"
+F 0 "#PWR084" H 5800 4550 30  0001 C CNN
 F 1 "GND" H 5800 4480 30  0001 C CNN
 	1    5800 4550
@@
 AR Path="/4FDB3935/4FDB29FE" Ref="R68"  Part="1"
 AR Path="/4FDB3936/4FDB29FE" Ref="R72"  Part="1"
-F 0 "R12" V 5130 3600 50  0000 C CNN
+F 0 "R72" V 5130 3600 50  0000 C CNN
 F 1 "2k4" V 5050 3600 50  0000 C CNN
 	1    5050 3600
@@
 AR Path="/4FDB3935/4FDB29E5" Ref="R67"  Part="1"
 AR Path="/4FDB3936/4FDB29E5" Ref="R71"  Part="1"
-F 0 "R11" V 4680 4250 50  0000 C CNN
+F 0 "R71" V 4680 4250 50  0000 C CNN
 F 1 "33k" V 4600 4250 50  0000 C CNN
 	1    4600 4250
@@
 AR Path="/4FDB3935/4FDB29D2" Ref="Q19"  Part="1"
 AR Path="/4FDB3936/4FDB29D2" Ref="Q20"  Part="1"
-F 0 "Q1" H 5700 3450 50  0000 R CNN
+F 0 "Q20" H 5700 3450 50  0000 R CNN
 F 1 "bc847" H 5700 3750 50  0000 R CNN
 	1    5700 3600

Commit message: SCH for motherboard is prepared. Power IO board is still not ready.
Changed lines of the file:
@@
-EESchema Schematic File Version 2  date Mon 18 Jun 2012 12:08:36 AM MSK
+EESchema Schematic File Version 2  date Mon 18 Jun 2012 01:18:32 AM MSK
 LIBS:power
 LIBS:device
@@
 Comment4 ""
 $EndDescr
-$Comp
-L VDD #PWR031
+Wire Wire Line
+	5800 2300 5800 2050
+Connection ~ 5800 3250
+Wire Wire Line
+	5800 3250 6250 3250
+Wire Wire Line
+	4600 4500 4600 4700
+Connection ~ 4600 3600
+Wire Wire Line
+	3900 3600 4800 3600
+Wire Wire Line
+	5300 3600 5500 3600
+Wire Wire Line
+	4600 3600 4600 4000
+Wire Wire Line
+	5800 3800 5800 4550
+Wire Wire Line
+	5800 3400 5800 2800
+Wire Wire Line
+	6750 3250 7150 3250
+$Comp
+L VDD #PWR014
 U 1 1 4FDB399C
 P 5800 2050
-AR Path="/4FDC7DE6/4FDB399C" Ref="#PWR031"  Part="1"
-AR Path="/4FDC7DE5/4FDB399C" Ref="#PWR034"  Part="1"
-AR Path="/4FDC7DE4/4FDB399C" Ref="#PWR037"  Part="1"
-AR Path="/4FDC7DE3/4FDB399C" Ref="#PWR040"  Part="1"
-AR Path="/4FDC7DB7/4FDB399C" Ref="#PWR043"  Part="1"
-AR Path="/4FDC7DB6/4FDB399C" Ref="#PWR046"  Part="1"
-AR Path="/4FDC7DB5/4FDB399C" Ref="#PWR049"  Part="1"
-AR Path="/4FDC7DB4/4FDB399C" Ref="#PWR052"  Part="1"
-AR Path="/4FDB299D/4FDB399C" Ref="#PWR073"  Part="1"
-AR Path="/4FDB3921/4FDB399C" Ref="#PWR076"  Part="1"
-AR Path="/4FDB3935/4FDB399C" Ref="#PWR079"  Part="1"
-AR Path="/4FDB3936/4FDB399C" Ref="#PWR082"  Part="1"
-F 0 "#PWR082" H 5800 2150 30  0001 C CNN
+AR Path="/4FDC7DE6/4FDB399C" Ref="#PWR014"  Part="1"
+AR Path="/4FDC7DE5/4FDB399C" Ref="#PWR017"  Part="1"
+AR Path="/4FDC7DE4/4FDB399C" Ref="#PWR020"  Part="1"
+AR Path="/4FDC7DE3/4FDB399C" Ref="#PWR023"  Part="1"
+AR Path="/4FDC7DB7/4FDB399C" Ref="#PWR026"  Part="1"
+AR Path="/4FDC7DB6/4FDB399C" Ref="#PWR029"  Part="1"
+AR Path="/4FDC7DB5/4FDB399C" Ref="#PWR032"  Part="1"
+AR Path="/4FDC7DB4/4FDB399C" Ref="#PWR035"  Part="1"
+AR Path="/4FDB299D/4FDB399C" Ref="#PWR056"  Part="1"
+AR Path="/4FDB3921/4FDB399C" Ref="#PWR059"  Part="1"
+AR Path="/4FDB3935/4FDB399C" Ref="#PWR062"  Part="1"
+AR Path="/4FDB3936/4FDB399C" Ref="#PWR065"  Part="1"
+F 0 "#PWR065" H 5800 2150 30  0001 C CNN
 F 1 "VDD" H 5800 2160 30  0000 C CNN
 	1    5800 2050
 	1    0    0    -1
 $EndComp
-Wire Wire Line
-	5800 2300 5800 2050
-Connection ~ 5800 3250
-Wire Wire Line
-	5800 3250 6250 3250
-Wire Wire Line
-	4600 4500 4600 4700
-Connection ~ 4600 3600
-Wire Wire Line
-	3900 3600 4800 3600
-Wire Wire Line
-	5300 3600 5500 3600
-Wire Wire Line
-	4600 3600 4600 4000
-Wire Wire Line
-	5800 3800 5800 4550
-Wire Wire Line
-	5800 3400 5800 2800
-Wire Wire Line
-	6750 3250 7150 3250
 $Comp
 L R R13
@@
 AR Path="/4FDB3935/4FDB2AE7" Ref="R69"  Part="1"
 AR Path="/4FDB3936/4FDB2AE7" Ref="R73"  Part="1"
-F 0 "R73" V 5880 2550 50  0000 C CNN
+F 0 "R13" V 5880 2550 50  0000 C CNN
 F 1 "33k" V 5800 2550 50  0000 C CNN
 	1    5800 2550
@@
 AR Path="/4FDB3935/4FDB2AA4" Ref="R70"  Part="1"
 AR Path="/4FDB3936/4FDB2AA4" Ref="R74"  Part="1"
-F 0 "R74" V 6580 3250 50  0000 C CNN
+F 0 "R14" V 6580 3250 50  0000 C CNN
 F 1 "2k4" V 6500 3250 50  0000 C CNN
 	1    6500 3250
@@
 $EndComp
 $Comp
-L GND #PWR032
+L GND #PWR015
 U 1 1 4FDB2A6B
 P 4600 4700
-AR Path="/4FDC7DE6/4FDB2A6B" Ref="#PWR032"  Part="1"
-AR Path="/4FDC7DE5/4FDB2A6B" Ref="#PWR035"  Part="1"
-AR Path="/4FDC7DE4/4FDB2A6B" Ref="#PWR038"  Part="1"
-AR Path="/4FDC7DE3/4FDB2A6B" Ref="#PWR041"  Part="1"
-AR Path="/4FDC7DB7/4FDB2A6B" Ref="#PWR044"  Part="1"
-AR Path="/4FDC7DB6/4FDB2A6B" Ref="#PWR047"  Part="1"
-AR Path="/4FDC7DB5/4FDB2A6B" Ref="#PWR050"  Part="1"
-AR Path="/4FDC7DB4/4FDB2A6B" Ref="#PWR053"  Part="1"
-AR Path="/4FDB299D/4FDB2A6B" Ref="#PWR074"  Part="1"
-AR Path="/4FDB3921/4FDB2A6B" Ref="#PWR077"  Part="1"
-AR Path="/4FDB3935/4FDB2A6B" Ref="#PWR080"  Part="1"
-AR Path="/4FDB3936/4FDB2A6B" Ref="#PWR083"  Part="1"
-F 0 "#PWR083" H 4600 4700 30  0001 C CNN
+AR Path="/4FDC7DE6/4FDB2A6B" Ref="#PWR015"  Part="1"
+AR Path="/4FDC7DE5/4FDB2A6B" Ref="#PWR018"  Part="1"
+AR Path="/4FDC7DE4/4FDB2A6B" Ref="#PWR021"  Part="1"
+AR Path="/4FDC7DE3/4FDB2A6B" Ref="#PWR024"  Part="1"
+AR Path="/4FDC7DB7/4FDB2A6B" Ref="#PWR027"  Part="1"
+AR Path="/4FDC7DB6/4FDB2A6B" Ref="#PWR030"  Part="1"
+AR Path="/4FDC7DB5/4FDB2A6B" Ref="#PWR033"  Part="1"
+AR Path="/4FDC7DB4/4FDB2A6B" Ref="#PWR036"  Part="1"
+AR Path="/4FDB299D/4FDB2A6B" Ref="#PWR057"  Part="1"
+AR Path="/4FDB3921/4FDB2A6B" Ref="#PWR060"  Part="1"
+AR Path="/4FDB3935/4FDB2A6B" Ref="#PWR063"  Part="1"
+AR Path="/4FDB3936/4FDB2A6B" Ref="#PWR066"  Part="1"
+F 0 "#PWR066" H 4600 4700 30  0001 C CNN
 F 1 "GND" H 4600 4630 30  0001 C CNN
 	1    4600 4700
@@
 $EndComp
 $Comp
-L GND #PWR033
+L GND #PWR016
 U 1 1 4FDB2A62
 P 5800 4550
-AR Path="/4FDC7DE6/4FDB2A62" Ref="#PWR033"  Part="1"
-AR Path="/4FDC7DE5/4FDB2A62" Ref="#PWR036"  Part="1"
-AR Path="/4FDC7DE4/4FDB2A62" Ref="#PWR039"  Part="1"
-AR Path="/4FDC7DE3/4FDB2A62" Ref="#PWR042"  Part="1"
-AR Path="/4FDC7DB7/4FDB2A62" Ref="#PWR045"  Part="1"
-AR Path="/4FDC7DB6/4FDB2A62" Ref="#PWR048"  Part="1"
-AR Path="/4FDC7DB5/4FDB2A62" Ref="#PWR051"  Part="1"
-AR Path="/4FDC7DB4/4FDB2A62" Ref="#PWR054"  Part="1"
-AR Path="/4FDB299D/4FDB2A62" Ref="#PWR075"  Part="1"
-AR Path="/4FDB3921/4FDB2A62" Ref="#PWR078"  Part="1"
-AR Path="/4FDB3935/4FDB2A62" Ref="#PWR081"  Part="1"
-AR Path="/4FDB3936/4FDB2A62" Ref="#PWR084"  Part="1"
-F 0 "#PWR084" H 5800 4550 30  0001 C CNN
+AR Path="/4FDC7DE6/4FDB2A62" Ref="#PWR016"  Part="1"
+AR Path="/4FDC7DE5/4FDB2A62" Ref="#PWR019"  Part="1"
+AR Path="/4FDC7DE4/4FDB2A62" Ref="#PWR022"  Part="1"
+AR Path="/4FDC7DE3/4FDB2A62" Ref="#PWR025"  Part="1"
+AR Path="/4FDC7DB7/4FDB2A62" Ref="#PWR028"  Part="1"
+AR Path="/4FDC7DB6/4FDB2A62" Ref="#PWR031"  Part="1"
+AR Path="/4FDC7DB5/4FDB2A62" Ref="#PWR034"  Part="1"
+AR Path="/4FDC7DB4/4FDB2A62" Ref="#PWR037"  Part="1"
+AR Path="/4FDB299D/4FDB2A62" Ref="#PWR058"  Part="1"
+AR Path="/4FDB3921/4FDB2A62" Ref="#PWR061"  Part="1"
+AR Path="/4FDB3935/4FDB2A62" Ref="#PWR064"  Part="1"
+AR Path="/4FDB3936/4FDB2A62" Ref="#PWR067"  Part="1"
+F 0 "#PWR067" H 5800 4550 30  0001 C CNN
 F 1 "GND" H 5800 4480 30  0001 C CNN
 	1    5800 4550
@@
 AR Path="/4FDB3935/4FDB29FE" Ref="R68"  Part="1"
 AR Path="/4FDB3936/4FDB29FE" Ref="R72"  Part="1"
-F 0 "R72" V 5130 3600 50  0000 C CNN
+F 0 "R12" V 5130 3600 50  0000 C CNN
 F 1 "2k4" V 5050 3600 50  0000 C CNN
 	1    5050 3600
@@
 AR Path="/4FDB3935/4FDB29E5" Ref="R67"  Part="1"
 AR Path="/4FDB3936/4FDB29E5" Ref="R71"  Part="1"
-F 0 "R71" V 4680 4250 50  0000 C CNN
+F 0 "R11" V 4680 4250 50  0000 C CNN
 F 1 "33k" V 4600 4250 50  0000 C CNN
 	1    4600 4250
@@
 AR Path="/4FDB3935/4FDB29D2" Ref="Q19"  Part="1"
 AR Path="/4FDB3936/4FDB29D2" Ref="Q20"  Part="1"
-F 0 "Q20" H 5700 3450 50  0000 R CNN
+F 0 "Q1" H 5700 3450 50  0000 R CNN
 F 1 "bc847" H 5700 3750 50  0000 R CNN
 	1    5700 3600
