File: schema/valve-power/output2.sch (KiCad schematic (older format))
At the start: 9 parts, among them Q4 MOSFET_N, Q5 MOSFET_N, U4 MC34152

Commit message: Valve-power board is in progress.
Parts:
- renumbered Q5 to Q10, Q4 to Q9, R46 to R43, R45 to R44, R36 to R45, R37 to R46, U4 to U3
Other:
- moved on the sheet: R51, R52
Changed lines of the file:
@@
-EESchema Schematic File Version 2  date Sat 16 Jun 2012 04:56:37 PM MSK
+EESchema Schematic File Version 2  date Sat 16 Jun 2012 11:30:21 PM MSK
 LIBS:power
 LIBS:device
@@
 $Descr A4 11700 8267
 encoding utf-8
-Sheet 6 17
+Sheet 12 17
 Title ""
 Date "16 jun 2012"
@@
 $EndDescr
 $Comp
-L GND #PWR058
-U 1 1 4FDC4E02
-P 9500 3050
-AR Path="/4FDB33F6/4FDC4E02" Ref="#PWR058"  Part="1"
-AR Path="/4FDB2BC5/4FDC4E02" Ref="#PWR063"  Part="1"
-F 0 "#PWR063" H 9500 3050 30  0001 C CNN
-F 1 "GND" H 9500 2980 30  0001 C CNN
-	1    9500 3050
-	1    0    0    -1
-$EndComp
-Wire Wire Line
-	9500 2950 9500 3050
-Wire Wire Line
-	7000 2900 7000 3000
+L GND #PWR054
+U 1 1 4FDCD69E
+P 4700 4900
+AR Path="/4FDC7CDA/4FDCD69E" Ref="#PWR054"  Part="1"
+AR Path="/4FDC7CD9/4FDCD69E" Ref="#PWR059"  Part="1"
+AR Path="/4FDB2BC5/4FDCD69E" Ref="#PWR025"  Part="1"
+AR Path="/4FDB33F6/4FDCD69E" Ref="#PWR064"  Part="1"
+F 0 "#PWR064" H 4700 4900 30  0001 C CNN
+F 1 "GND" H 4700 4830 30  0001 C CNN
+	1    4700 4900
+	1    0    0    -1
+$EndComp
+Wire Wire Line
+	5000 4700 5000 4900
+Connection ~ 4700 3550
+Wire Wire Line
+	4700 4200 4700 3550
 Wire Wire Line
 	5800 4400 5800 4900
@@
 Connection ~ 9900 1800
 Wire Wire Line
-	7000 2400 7000 2100
-Connection ~ 7000 2100
-Wire Wire Line
-	9500 2450 9500 2100
-Connection ~ 9500 2100
-$Comp
-L R R45
+	5000 4200 5000 4000
+Connection ~ 5000 4000
+Wire Wire Line
+	4700 4700 4700 4900
+$Comp
+L GND #PWR055
+U 1 1 4FDC4E02
+P 5000 4900
+AR Path="/4FDC7CDA/4FDC4E02" Ref="#PWR055"  Part="1"
+AR Path="/4FDC7CD9/4FDC4E02" Ref="#PWR060"  Part="1"
+AR Path="/4FDB2BC5/4FDC4E02" Ref="#PWR026"  Part="1"
+AR Path="/4FDB33F6/4FDC4E02" Ref="#PWR065"  Part="1"
+F 0 "#PWR065" H 5000 4900 30  0001 C CNN
+F 1 "GND" H 5000 4830 30  0001 C CNN
+	1    5000 4900
+	1    0    0    -1
+$EndComp
+$Comp
+L R R44
 U 1 1 4FDC4DF4
-P 9500 2700
-AR Path="/4FDB33F6/4FDC4DF4" Ref="R45"  Part="1"
-AR Path="/4FDB2BC5/4FDC4DF4" Ref="R47"  Part="1"
-F 0 "R47" V 9580 2700 50  0000 C CNN
-F 1 "33k" V 9500 2700 50  0000 C CNN
-	1    9500 2700
+P 5000 4450
+AR Path="/4FDC7CDA/4FDC4DF4" Ref="R44"  Part="1"
+AR Path="/4FDC7CD9/4FDC4DF4" Ref="R48"  Part="1"
+AR Path="/4FDB2BC5/4FDC4DF4" Ref="R52"  Part="1"
+AR Path="/4FDB33F6/4FDC4DF4" Ref="R56"  Part="1"
+F 0 "R52" V 5080 4450 50  0000 C CNN
+F 1 "33k" V 5000 4450 50  0000 C CNN
+	1    5000 4450
 	-1   0    0    1
 $EndComp
 $Comp
-L GND #PWR059
-U 1 1 4FDC4DE7
-P 7000 3000
-AR Path="/4FDB33F6/4FDC4DE7" Ref="#PWR059"  Part="1"
-AR Path="/4FDB2BC5/4FDC4DE7" Ref="#PWR064"  Part="1"
-F 0 "#PWR064" H 7000 3000 30  0001 C CNN
-F 1 "GND" H 7000 2930 30  0001 C CNN
-	1    7000 3000
-	1    0    0    -1
-$EndComp
-$Comp
-L R R46
+L R R43
 U 1 1 4FDC4DD8
-P 7000 2650
-AR Path="/4FDB2BC5/4FDC4DD8" Ref="R46"  Part="1"
-AR Path="/4FDB33F6/4FDC4DD8" Ref="R44"  Part="1"
-F 0 "R46" V 7080 2650 50  0000 C CNN
-F 1 "33k" V 7000 2650 50  0000 C CNN
-	1    7000 2650
+P 4700 4450
+AR Path="/4FDC7CDA/4FDC4DD8" Ref="R43"  Part="1"
+AR Path="/4FDC7CD9/4FDC4DD8" Ref="R47"  Part="1"
+AR Path="/4FDB2BC5/4FDC4DD8" Ref="R51"  Part="1"
+AR Path="/4FDB33F6/4FDC4DD8" Ref="R55"  Part="1"
+F 0 "R51" V 4780 4450 50  0000 C CNN
+F 1 "33k" V 4700 4450 50  0000 C CNN
+	1    4700 4450
 	-1   0    0    1
 $EndComp
@@
 NoConn ~ 5100 3150
 $Comp
-L GND #PWR060
+L GND #PWR056
 U 1 1 4FDB2F05
 P 5800 4900
-AR Path="/4FDB33F6/4FDB2F05" Ref="#PWR060"  Part="1"
-AR Path="/4FDB2BC5/4FDB2F05" Ref="#PWR065"  Part="1"
-F 0 "#PWR065" H 5800 4900 30  0001 C CNN
+AR Path="/4FDC7CDA/4FDB2F05" Ref="#PWR056"  Part="1"
+AR Path="/4FDC7CD9/4FDB2F05" Ref="#PWR061"  Part="1"
+AR Path="/4FDB2BC5/4FDB2F05" Ref="#PWR027"  Part="1"
+AR Path="/4FDB33F6/4FDB2F05" Ref="#PWR066"  Part="1"
+F 0 "#PWR066" H 5800 4900 30  0001 C CNN
 F 1 "GND" H 5800 4830 30  0001 C CNN
 	1    5800 4900
@@
 outA
 $Comp
-L R R37
+L R R46
 U 1 1 4FDB2ED0
 P 9150 2100
-AR Path="/4FDB33F6/4FDB2ED0" Ref="R37"  Part="1"
-AR Path="/4FDB2BC5/4FDB2ED0" Ref="R39"  Part="1"
-F 0 "R39" V 9230 2100 50  0000 C CNN
+AR Path="/4FDC7CDA/4FDB2ED0" Ref="R46"  Part="1"
+AR Path="/4FDC7CD9/4FDB2ED0" Ref="R50"  Part="1"
+AR Path="/4FDB2BC5/4FDB2ED0" Ref="R54"  Part="1"
+AR Path="/4FDB33F6/4FDB2ED0" Ref="R58"  Part="1"
+F 0 "R54" V 9230 2100 50  0000 C CNN
 F 1 "10" V 9150 2100 50  0000 C CNN
 	1    9150 2100
@@
 $EndComp
 $Comp
-L MOSFET_N Q5
+L MOSFET_N Q10
 U 1 1 4FDB2ECF
 P 9800 2100
-AR Path="/4FDB33F6/4FDB2ECF" Ref="Q5"  Part="1"
-AR Path="/4FDB2BC5/4FDB2ECF" Ref="Q7"  Part="1"
-F 0 "Q7" H 9810 2270 60  0000 R CNN
+AR Path="/4FDC7CDA/4FDB2ECF" Ref="Q10"  Part="1"
+AR Path="/4FDC7CD9/4FDB2ECF" Ref="Q12"  Part="1"
+AR Path="/4FDB2BC5/4FDB2ECF" Ref="Q14"  Part="1"
+AR Path="/4FDB33F6/4FDB2ECF" Ref="Q16"  Part="1"
+F 0 "Q14" H 9810 2270 60  0000 R CNN
 F 1 "MOSFET_N" H 9810 1950 60  0000 R CNN
 	1    9800 2100
@@
 $EndComp
 $Comp
-L GND #PWR061
+L GND #PWR057
 U 1 1 4FDB2ECE
 P 9900 2550
-AR Path="/4FDB33F6/4FDB2ECE" Ref="#PWR061"  Part="1"
-AR Path="/4FDB2BC5/4FDB2ECE" Ref="#PWR066"  Part="1"
-F 0 "#PWR066" H 9900 2550 30  0001 C CNN
+AR Path="/4FDC7CDA/4FDB2ECE" Ref="#PWR057"  Part="1"
+AR Path="/4FDC7CD9/4FDB2ECE" Ref="#PWR062"  Part="1"
+AR Path="/4FDB2BC5/4FDB2ECE" Ref="#PWR028"  Part="1"
+AR Path="/4FDB33F6/4FDB2ECE" Ref="#PWR067"  Part="1"
+F 0 "#PWR067" H 9900 2550 30  0001 C CNN
 F 1 "GND" H 9900 2480 30  0001 C CNN
 	1    9900 2550
@@
 U 1 1 4FDB2ECD
 P 9900 1500
-AR Path="/4FDB33F6/4FDB2ECD" Ref="D4"  Part="1"
-AR Path="/4FDB2BC5/4FDB2ECD" Ref="D6"  Part="1"
-F 0 "D6" H 9900 1600 40  0000 C CNN
+AR Path="/4FDC7CDA/4FDB2ECD" Ref="D4"  Part="1"
+AR Path="/4FDC7CD9/4FDB2ECD" Ref="D6"  Part="1"
+AR Path="/4FDB2BC5/4FDB2ECD" Ref="D8"  Part="1"
+AR Path="/4FDB33F6/4FDB2ECD" Ref="D10"  Part="1"
+F 0 "D8" H 9900 1600 40  0000 C CNN
 F 1 "1N4148" H 9900 1400 40  0000 C CNN
 	1    9900 1500
@@
 U 1 1 4FDB2DC3
 P 7400 1500
-AR Path="/4FDB33F6/4FDB2DC3" Ref="D3"  Part="1"
-AR Path="/4FDB2BC5/4FDB2DC3" Ref="D5"  Part="1"
-F 0 "D5" H 7400 1600 40  0000 C CNN
+AR Path="/4FDC7CDA/4FDB2DC3" Ref="D3"  Part="1"
+AR Path="/4FDC7CD9/4FDB2DC3" Ref="D5"  Part="1"
+AR Path="/4FDB2BC5/4FDB2DC3" Ref="D7"  Part="1"
+AR Path="/4FDB33F6/4FDB2DC3" Ref="D9"  Part="1"
+F 0 "D7" H 7400 1600 40  0000 C CNN
 F 1 "1N4148" H 7400 1400 40  0000 C CNN
 	1    7400 1500
@@
 $EndComp
 $Comp
-L GND #PWR062
+L GND #PWR058
 U 1 1 4FDB2D3E
 P 7400 2550
-AR Path="/4FDB33F6/4FDB2D3E" Ref="#PWR062"  Part="1"
-AR Path="/4FDB2BC5/4FDB2D3E" Ref="#PWR067"  Part="1"
-F 0 "#PWR067" H 7400 2550 30  0001 C CNN
+AR Path="/4FDC7CDA/4FDB2D3E" Ref="#PWR058"  Part="1"
+AR Path="/4FDC7CD9/4FDB2D3E" Ref="#PWR063"  Part="1"
+AR Path="/4FDB2BC5/4FDB2D3E" Ref="#PWR029"  Part="1"
+AR Path="/4FDB33F6/4FDB2D3E" Ref="#PWR068"  Part="1"
+F 0 "#PWR068" H 7400 2550 30  0001 C CNN
 F 1 "GND" H 7400 2480 30  0001 C CNN
 	1    7400 2550
@@
 $EndComp
 $Comp
-L MOSFET_N Q4
+L MOSFET_N Q9
 U 1 1 4FDB2C4B
 P 7300 2100
-AR Path="/4FDB33F6/4FDB2C4B" Ref="Q4"  Part="1"
-AR Path="/4FDB2BC5/4FDB2C4B" Ref="Q6"  Part="1"
-F 0 "Q6" H 7310 2270 60  0000 R CNN
+AR Path="/4FDC7CDA/4FDB2C4B" Ref="Q9"  Part="1"
+AR Path="/4FDC7CD9/4FDB2C4B" Ref="Q11"  Part="1"
+AR Path="/4FDB2BC5/4FDB2C4B" Ref="Q13"  Part="1"
+AR Path="/4FDB33F6/4FDB2C4B" Ref="Q15"  Part="1"
+F 0 "Q13" H 7310 2270 60  0000 R CNN
 F 1 "MOSFET_N" H 7310 1950 60  0000 R CNN
 	1    7300 2100
@@
 $EndComp
 $Comp
-L R R36
+L R R45
 U 1 1 4FDB2C18
 P 6650 2100
-AR Path="/4FDB33F6/4FDB2C18" Ref="R36"  Part="1"
-AR Path="/4FDB2BC5/4FDB2C18" Ref="R38"  Part="1"
-F 0 "R38" V 6730 2100 50  0000 C CNN
+AR Path="/4FDC7CDA/4FDB2C18" Ref="R45"  Part="1"
+AR Path="/4FDC7CD9/4FDB2C18" Ref="R49"  Part="1"
+AR Path="/4FDB2BC5/4FDB2C18" Ref="R53"  Part="1"
+AR Path="/4FDB33F6/4FDB2C18" Ref="R57"  Part="1"
+F 0 "R53" V 6730 2100 50  0000 C CNN
 F 1 "10" V 6650 2100 50  0000 C CNN
 	1    6650 2100
@@
 $EndComp
 $Comp
-L MC34152 U4
+L MC34152 U3
 U 1 1 4FDB2BFB
 P 5800 3750
-AR Path="/4FDB33F6/4FDB2BFB" Ref="U4"  Part="1"
+AR Path="/4FDC7CDA/4FDB2BFB" Ref="U3"  Part="1"
+AR Path="/4FDC7CD9/4FDB2BFB" Ref="U4"  Part="1"
 AR Path="/4FDB2BC5/4FDB2BFB" Ref="U5"  Part="1"
+AR Path="/4FDB33F6/4FDB2BFB" Ref="U6"  Part="1"
 F 0 "U5" H 5800 4100 60  0000 C CNN
 F 1 "MC34152" H 5800 3750 60  0000 C CNN
