File: schema/valve-power/output2.sch (KiCad schematic (older format))
At the start: 9 parts, among them Q10 MOSFET_N, Q9 MOSFET_N, U3 MC34152

Commit message: Power supply board is ready.
Parts:
- added C11: 100n, symbol C
Connections:
- wire segments 22 -> 24
Other:
- note added: "Gate supply filtering because \nit comes through long wires."
Changed lines of the file:
@@
-EESchema Schematic File Version 2  date Sun 17 Jun 2012 09:58:46 PM MSK
+EESchema Schematic File Version 2  date Mon 18 Jun 2012 12:08:36 AM MSK
 LIBS:power
 LIBS:device
@@
 $Descr A4 11700 8267
 encoding utf-8
-Sheet 11 17
+Sheet 2 17
 Title ""
 Date "17 jun 2012"
@@
 Comment4 ""
 $EndDescr
-$Comp
-L GND #PWR054
+Text Notes 4150 2550 1    60   ~ 0
+Gate supply filtering because \nit comes through long wires.
+Text GLabel 4500 1500 1    60   Input ~ 0
+10V
+$Comp
+L GND #PWR025
+U 1 1 4FDE3727
+P 4500 2500
+AR Path="/4FDB2BC5/4FDE3727" Ref="#PWR025"  Part="1"
+AR Path="/4FDC7CDA/4FDE3727" Ref="#PWR055"  Part="1"
+AR Path="/4FDC7CD9/4FDE3727" Ref="#PWR061"  Part="1"
+AR Path="/4FDB33F6/4FDE3727" Ref="#PWR067"  Part="1"
+F 0 "#PWR025" H 4500 2500 30  0001 C CNN
+F 1 "GND" H 4500 2430 30  0001 C CNN
+	1    4500 2500
+	1    0    0    -1
+$EndComp
+Wire Wire Line
+	4500 2200 4500 2500
+Wire Wire Line
+	5000 4700 5000 4900
+Connection ~ 4700 3550
+Wire Wire Line
+	4700 4200 4700 3550
+Wire Wire Line
+	5800 4400 5800 4900
+Connection ~ 7400 1800
+Wire Wire Line
+	7400 1800 8300 1800
+Wire Wire Line
+	7400 1900 7400 1700
+Wire Wire Line
+	6400 2100 6200 2100
+Wire Wire Line
+	6550 4000 7100 4000
+Wire Wire Line
+	5100 4000 4500 4000
+Wire Wire Line
+	5100 3550 4500 3550
+Wire Wire Line
+	6550 3550 7100 3550
+Wire Wire Line
+	7100 2100 6900 2100
+Wire Wire Line
+	7400 2300 7400 2550
+Wire Wire Line
+	7400 1300 7400 950
+Wire Wire Line
+	5800 2750 5800 2250
+Wire Wire Line
+	9900 1300 9900 950
+Wire Wire Line
+	9900 2300 9900 2550
+Wire Wire Line
+	9600 2100 9400 2100
+Wire Wire Line
+	8900 2100 8700 2100
+Wire Wire Line
+	9900 1900 9900 1700
+Wire Wire Line
+	9900 1800 10800 1800
+Connection ~ 9900 1800
+Wire Wire Line
+	5000 4200 5000 4000
+Connection ~ 5000 4000
+Wire Wire Line
+	4700 4700 4700 4900
+Wire Wire Line
+	4500 1800 4500 1500
+$Comp
+L C C11
+U 1 1 4FDE3711
+P 4500 2000
+AR Path="/4FDB2BC5/4FDE3711" Ref="C11"  Part="1"
+AR Path="/4FDC7CDA/4FDE3711" Ref="C12"  Part="1"
+AR Path="/4FDC7CD9/4FDE3711" Ref="C13"  Part="1"
+AR Path="/4FDB33F6/4FDE3711" Ref="C14"  Part="1"
+F 0 "C11" H 4550 2100 50  0000 L CNN
+F 1 "100n" H 4550 1900 50  0000 L CNN
+	1    4500 2000
+	1    0    0    -1
+$EndComp
+$Comp
+L GND #PWR056
 U 1 1 4FDCD69E
 P 4700 4900
-AR Path="/4FDC7CDA/4FDCD69E" Ref="#PWR054"  Part="1"
-AR Path="/4FDC7CD9/4FDCD69E" Ref="#PWR059"  Part="1"
-AR Path="/4FDB2BC5/4FDCD69E" Ref="#PWR025"  Part="1"
-AR Path="/4FDB33F6/4FDCD69E" Ref="#PWR064"  Part="1"
-F 0 "#PWR064" H 4700 4900 30  0001 C CNN
+AR Path="/4FDC7CDA/4FDCD69E" Ref="#PWR056"  Part="1"
+AR Path="/4FDC7CD9/4FDCD69E" Ref="#PWR062"  Part="1"
+AR Path="/4FDB2BC5/4FDCD69E" Ref="#PWR026"  Part="1"
+AR Path="/4FDB33F6/4FDCD69E" Ref="#PWR068"  Part="1"
+F 0 "#PWR026" H 4700 4900 30  0001 C CNN
 F 1 "GND" H 4700 4830 30  0001 C CNN
 	1    4700 4900
 	1    0    0    -1
 $EndComp
-Wire Wire Line
-	5000 4700 5000 4900
-Connection ~ 4700 3550
-Wire Wire Line
-	4700 4200 4700 3550
-Wire Wire Line
-	5800 4400 5800 4900
-Connection ~ 7400 1800
-Wire Wire Line
-	7400 1800 8300 1800
-Wire Wire Line
-	7400 1900 7400 1700
-Wire Wire Line
-	6400 2100 6200 2100
-Wire Wire Line
-	6550 4000 7100 4000
-Wire Wire Line
-	5100 4000 4500 4000
-Wire Wire Line
-	5100 3550 4500 3550
-Wire Wire Line
-	6550 3550 7100 3550
-Wire Wire Line
-	7100 2100 6900 2100
-Wire Wire Line
-	7400 2300 7400 2550
-Wire Wire Line
-	7400 1300 7400 950
-Wire Wire Line
-	5800 2750 5800 2250
-Wire Wire Line
-	9900 1300 9900 950
-Wire Wire Line
-	9900 2300 9900 2550
-Wire Wire Line
-	9600 2100 9400 2100
-Wire Wire Line
-	8900 2100 8700 2100
-Wire Wire Line
-	9900 1900 9900 1700
-Wire Wire Line
-	9900 1800 10800 1800
-Connection ~ 9900 1800
-Wire Wire Line
-	5000 4200 5000 4000
-Connection ~ 5000 4000
-Wire Wire Line
-	4700 4700 4700 4900
-$Comp
-L GND #PWR055
+$Comp
+L GND #PWR057
 U 1 1 4FDC4E02
 P 5000 4900
-AR Path="/4FDC7CDA/4FDC4E02" Ref="#PWR055"  Part="1"
-AR Path="/4FDC7CD9/4FDC4E02" Ref="#PWR060"  Part="1"
-AR Path="/4FDB2BC5/4FDC4E02" Ref="#PWR026"  Part="1"
-AR Path="/4FDB33F6/4FDC4E02" Ref="#PWR065"  Part="1"
-F 0 "#PWR065" H 5000 4900 30  0001 C CNN
+AR Path="/4FDC7CDA/4FDC4E02" Ref="#PWR057"  Part="1"
+AR Path="/4FDC7CD9/4FDC4E02" Ref="#PWR063"  Part="1"
+AR Path="/4FDB2BC5/4FDC4E02" Ref="#PWR027"  Part="1"
+AR Path="/4FDB33F6/4FDC4E02" Ref="#PWR069"  Part="1"
+F 0 "#PWR027" H 5000 4900 30  0001 C CNN
 F 1 "GND" H 5000 4830 30  0001 C CNN
 	1    5000 4900
@@
 AR Path="/4FDB2BC5/4FDC4DF4" Ref="R52"  Part="1"
 AR Path="/4FDB33F6/4FDC4DF4" Ref="R56"  Part="1"
-F 0 "R44" V 5080 4450 50  0000 C CNN
+F 0 "R52" V 5080 4450 50  0000 C CNN
 F 1 "33k" V 5000 4450 50  0000 C CNN
 	1    5000 4450
@@
 AR Path="/4FDB2BC5/4FDC4DD8" Ref="R51"  Part="1"
 AR Path="/4FDB33F6/4FDC4DD8" Ref="R55"  Part="1"
-F 0 "R43" V 4780 4450 50  0000 C CNN
+F 0 "R51" V 4780 4450 50  0000 C CNN
 F 1 "33k" V 4700 4450 50  0000 C CNN
 	1    4700 4450
@@
 NoConn ~ 5100 3150
 $Comp
-L GND #PWR056
+L GND #PWR058
 U 1 1 4FDB2F05
 P 5800 4900
-AR Path="/4FDC7CDA/4FDB2F05" Ref="#PWR056"  Part="1"
-AR Path="/4FDC7CD9/4FDB2F05" Ref="#PWR061"  Part="1"
-AR Path="/4FDB2BC5/4FDB2F05" Ref="#PWR027"  Part="1"
-AR Path="/4FDB33F6/4FDB2F05" Ref="#PWR066"  Part="1"
-F 0 "#PWR066" H 5800 4900 30  0001 C CNN
+AR Path="/4FDC7CDA/4FDB2F05" Ref="#PWR058"  Part="1"
+AR Path="/4FDC7CD9/4FDB2F05" Ref="#PWR064"  Part="1"
+AR Path="/4FDB2BC5/4FDB2F05" Ref="#PWR028"  Part="1"
+AR Path="/4FDB33F6/4FDB2F05" Ref="#PWR070"  Part="1"
+F 0 "#PWR028" H 5800 4900 30  0001 C CNN
 F 1 "GND" H 5800 4830 30  0001 C CNN
 	1    5800 4900
@@
 AR Path="/4FDB2BC5/4FDB2ED0" Ref="R54"  Part="1"
 AR Path="/4FDB33F6/4FDB2ED0" Ref="R58"  Part="1"
-F 0 "R46" V 9230 2100 50  0000 C CNN
+F 0 "R54" V 9230 2100 50  0000 C CNN
 F 1 "10" V 9150 2100 50  0000 C CNN
 	1    9150 2100
@@
 AR Path="/4FDB2BC5/4FDB2ECF" Ref="Q14"  Part="1"
 AR Path="/4FDB33F6/4FDB2ECF" Ref="Q16"  Part="1"
-F 0 "Q10" H 9810 2270 60  0000 R CNN
+F 0 "Q14" H 9810 2270 60  0000 R CNN
 F 1 "MOSFET_N" H 9810 1950 60  0000 R CNN
 	1    9800 2100
@@
 $EndComp
 $Comp
-L GND #PWR057
+L GND #PWR059
 U 1 1 4FDB2ECE
 P 9900 2550
-AR Path="/4FDC7CDA/4FDB2ECE" Ref="#PWR057"  Part="1"
-AR Path="/4FDC7CD9/4FDB2ECE" Ref="#PWR062"  Part="1"
-AR Path="/4FDB2BC5/4FDB2ECE" Ref="#PWR028"  Part="1"
-AR Path="/4FDB33F6/4FDB2ECE" Ref="#PWR067"  Part="1"
-F 0 "#PWR067" H 9900 2550 30  0001 C CNN
+AR Path="/4FDC7CDA/4FDB2ECE" Ref="#PWR059"  Part="1"
+AR Path="/4FDC7CD9/4FDB2ECE" Ref="#PWR065"  Part="1"
+AR Path="/4FDB2BC5/4FDB2ECE" Ref="#PWR029"  Part="1"
+AR Path="/4FDB33F6/4FDB2ECE" Ref="#PWR071"  Part="1"
+F 0 "#PWR029" H 9900 2550 30  0001 C CNN
 F 1 "GND" H 9900 2480 30  0001 C CNN
 	1    9900 2550
@@
 AR Path="/4FDB2BC5/4FDB2ECD" Ref="D8"  Part="1"
 AR Path="/4FDB33F6/4FDB2ECD" Ref="D10"  Part="1"
-F 0 "D4" H 9900 1600 40  0000 C CNN
+F 0 "D8" H 9900 1600 40  0000 C CNN
 F 1 "1N4148" H 9900 1400 40  0000 C CNN
 	1    9900 1500
@@
 AR Path="/4FDB2BC5/4FDB2DC3" Ref="D7"  Part="1"
 AR Path="/4FDB33F6/4FDB2DC3" Ref="D9"  Part="1"
-F 0 "D3" H 7400 1600 40  0000 C CNN
+F 0 "D7" H 7400 1600 40  0000 C CNN
 F 1 "1N4148" H 7400 1400 40  0000 C CNN
 	1    7400 1500
@@
 $EndComp
 $Comp
-L GND #PWR058
+L GND #PWR060
 U 1 1 4FDB2D3E
 P 7400 2550
-AR Path="/4FDC7CDA/4FDB2D3E" Ref="#PWR058"  Part="1"
-AR Path="/4FDC7CD9/4FDB2D3E" Ref="#PWR063"  Part="1"
-AR Path="/4FDB2BC5/4FDB2D3E" Ref="#PWR029"  Part="1"
-AR Path="/4FDB33F6/4FDB2D3E" Ref="#PWR068"  Part="1"
-F 0 "#PWR068" H 7400 2550 30  0001 C CNN
+AR Path="/4FDC7CDA/4FDB2D3E" Ref="#PWR060"  Part="1"
+AR Path="/4FDC7CD9/4FDB2D3E" Ref="#PWR066"  Part="1"
+AR Path="/4FDB2BC5/4FDB2D3E" Ref="#PWR030"  Part="1"
+AR Path="/4FDB33F6/4FDB2D3E" Ref="#PWR072"  Part="1"
+F 0 "#PWR030" H 7400 2550 30  0001 C CNN
 F 1 "GND" H 7400 2480 30  0001 C CNN
 	1    7400 2550
@@
 AR Path="/4FDB2BC5/4FDB2C4B" Ref="Q13"  Part="1"
 AR Path="/4FDB33F6/4FDB2C4B" Ref="Q15"  Part="1"
-F 0 "Q9" H 7310 2270 60  0000 R CNN
+F 0 "Q13" H 7310 2270 60  0000 R CNN
 F 1 "MOSFET_N" H 7310 1950 60  0000 R CNN
 	1    7300 2100
@@
 AR Path="/4FDB2BC5/4FDB2C18" Ref="R53"  Part="1"
 AR Path="/4FDB33F6/4FDB2C18" Ref="R57"  Part="1"
-F 0 "R45" V 6730 2100 50  0000 C CNN
+F 0 "R53" V 6730 2100 50  0000 C CNN
 F 1 "10" V 6650 2100 50  0000 C CNN
 	1    6650 2100
@@
 AR Path="/4FDB2BC5/4FDB2BFB" Ref="U5"  Part="1"
 AR Path="/4FDB33F6/4FDB2BFB" Ref="U6"  Part="1"
-F 0 "U3" H 5800 4100 60  0000 C CNN
+F 0 "U5" H 5800 4100 60  0000 C CNN
 F 1 "MC34152" H 5800 3750 60  0000 C CNN
 	1    5800 3750
