File: schema/valve-power/valve-power.sch (KiCad schematic (older format))
At the start: 39 parts

Commit message: Силовая часть. Плата управления клапанами.
Parts:
- removed P? (x8): port-out, symbol CONN_2
- removed P? (x2): 10v, symbol CONN_2
- removed P?: 3.3v, symbol CONN_2
- added P?: CONN_12, symbol CONN_12
- added P?: CONN_8, symbol CONN_8
- added P?: CONN_20, symbol CONN_20
Connections:
- net labels added: in10, in11, in12, in5, in6, in7, in8, in9, io1, io10, io11, io12, io13, io14, io15, io16, io17, io18, io19, io2, io20, io3, io4, io5, io6, io7, io8, io9, out5, out6, out7, out8
- net labels removed: out-int1, out-int2, out-int3, out-int4
- wire segments 138 -> 170
Other:
- note added: "24v digital inputs"
- note added: "Digital IO board interaction sockets"
- note added: "Outputs for driving inductive load"
- note added: "Power IOs"
- moved on the sheet: P?

Commit message: Valve-power board is in progress.
Parts:
- added P6, P7, P8, P9: CONN_1, symbol CONN_1
- gave numbers to parts that had none: 31
Connections:
- no-connect marks 0 -> 4
Other:
- note added: "Mounting holes for screwing."
