File: schema/valve-power/valve-power.sch (KiCad schematic (older format))
At the start: 35 parts, among them P1 CONN_12, P2 CONN_8, P3 3.3v, P4 CONN_20, P5 24v, P6 CONN_1, P7 CONN_1, P8 CONN_1, P9 CONN_1, U1 NCP3063, U2 NCP3063

Commit message: SCH for motherboard is prepared. Power IO board is still not ready.
Parts:
- removed C1, C2: 4u7, symbol C
- removed C10, C9: 1m, symbol C
- removed C3, C4, C7, C8: 100n, symbol C
- removed C5, C6: 2.2n, symbol C
- removed D1, D2: 1N5819, symbol DIODESCH
- removed L1, L2: INDUCTOR, symbol INDUCTOR
- removed P1: CONN_12, symbol CONN_12
- removed P2: CONN_8, symbol CONN_8
- removed P3: 3.3v, symbol CONN_2
- removed P5: 24v, symbol CONN_4
- removed P6, P7, P8, P9: CONN_1, symbol CONN_1
- removed R1, R2, R3, R4, R5, R6: 1R5, symbol R
- removed R10: 50k, symbol R
- removed R7: 12k, symbol R
- removed R8: 10k, symbol R
- removed R9: 20k, symbol R
- removed U1, U2: NCP3063, symbol NCP3063
- added P1: CONN_20, symbol CONN_20
- added P2: CONN_6, symbol CONN_6
Connections:
- net labels removed: 10v-out, buck-out
- wire segments 170 -> 97
- no-connect marks 4 -> 0
Other:
- note removed: "Mounting holes for screwing."
