File: schema/valve_2/valve_2.sch (KiCad schematic (older format))
At the start: 48 parts

Commit message: Drawing valve control board 2-d revision.
Parts:
- added C?: 10u, symbol C
- added J? (x2): DB37, symbol DB37
- added R? (x20): 10k, symbol R
- added R? (x16): 1k5, symbol R
- added U? (x6): L293, symbol L293
Connections:
- net labels added: gnd, isock0, isock1, isock10, isock11, isock12, isock13, isock14, isock15, isock2, isock3, isock4, isock5, isock6, isock7, isock8, isock9, sock0, sock1, sock10, sock11, sock12, sock13, sock14, sock15, sock16, sock17, sock18, sock19, sock2, sock20, sock21, sock22, sock23, sock24, sock25, sock26, sock27, sock3, sock4, sock5, sock6, sock7, sock8, sock9
- wire segments 305 -> 573

Commit message: Drawing sockets.
Connections:
- net labels added: 24v
- wire segments 573 -> 621
