File: schema/valve_2/valve_2.sch (KiCad schematic (older format))
At the start: 114 parts, among them J1 DB37, J2 DB37, J3 DB9, P1 SETUP, P2 CROSS-BRD-1, P3 CROSS-BRD-2, P4 SWD-IAP, U1 74HC165, U10 L293, U11 L293, U12 L293, U13 L293, U14 MINI-USB-B, U15 NCP3063, U16 NCP3063, U2 74HC165, U3 74HC164, U4 74HC164, U5 74HC164, U6 74HC164, U7 L293, U8 L293, U9 L293, X1 8MHz

Commit message: Made separate I2C sockets couple close to MCU to minimize cross currents from other PCB parts.
Parts:
- removed C12, C17: 100n, symbol C
- removed P2: CROSS-BRD-1, symbol CONN_17
- removed P3: CROSS-BRD-2, symbol CONN_17
- added C? (x4): 10u, symbol C
- added K1: i2c-1, symbol CONN_3
- added K2: i2c-2, symbol CONN_3
- added P2: power-1, symbol CONN_12
- added P3: power-2, symbol CONN_12
- added R63, R64: 100, symbol R
Connections:
- net labels added: scl-ext, sda-ext
- wire segments 693 -> 689
Other:
- moved on the sheet: C10, C11, C13, C14, C15, C8, C9, D4, L1, R41, R42, R43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

Commit message: Routing...
Parts:
- gave numbers to parts that had none: 4

Commit message: Routing...
Other:
- note added: "dry switch"
- note added: "sdy switch\n"
- note added: "vac relay\n"
