File: schema/cable-executive/cable-executive.sch (KiCad schematic (older format))
At the start: 87 parts

Commit message: Drawing cables...
Parts:
- added Conn? (x2): D-SUB-37, symbol D-SUB-37
Connections:
- net connb-17: no longer Conn?.18
- net connb-18: no longer Conn?.19
- net connb-19: no longer Conn?.20
- net connb-20: no longer Conn?.21
- net connb-21: no longer Conn?.22
- net connb-22: no longer Conn?.23
- net connb-23: no longer Conn?.24
- net connb-24: no longer Conn?.25
- net connb-25: no longer Conn?.26
- net connb-26: no longer Conn?.27
- net connb-27: no longer Conn?.28
- net connb-28: no longer Conn?.29
- net connb-29: no longer Conn?.30
- net connb-30: no longer Conn?.31
- net connb-31: no longer Conn?.32
- net connb-32: no longer Conn?.33
- net connb-33: no longer Conn?.34
- net connb-34: no longer Conn?.35
- net connb-35: no longer Conn?.36
- net connb-36: no longer Conn?.37
- net connc-10: now also conn?.2
- net connc-11: now also conn?.3
- net connc-12: now also conn?.1
- net connc-13: now also conn?.2
- net connc-14: now also conn?.3
- net connc-15: now also conn?.1
- net connc-16: now also conn?.2
- net connc-17: now also conn?.3
- net connc-18: now also conn?.1
- net connc-19: now also conn?.2
- net connc-20: now also conn?.3
- net connc-21: now also conn?.1
- net connc-22: now also conn?.2
- net connc-23: now also conn?.3
- net connc-24: now also conn?.1
- net connc-25: now also conn?.2
- net connc-26: now also conn?.3
- net connc-27: now also conn?.1
- net connc-28: now also conn?.2
- net connc-29: now also conn?.3
- net connc-3: now also conn?.1
- net connc-30: now also conn?.1
- net connc-31: now also conn?.2
- net connc-32: now also conn?.3
- net connc-33: now also conn?.1
- net connc-34: now also conn?.2
- net connc-35: now also conn?.3
- net connc-4: now also conn?.2
- net connc-5: now also conn?.3
- net connc-6: now also conn?.1
- net connc-7: now also conn?.2
- net connc-8: now also conn?.3
- net connc-9: now also conn?.1
- net connd-0: now also conn?.1
- net connd-1: now also conn?.2
- net connd-10: now also switch?.2
- net connd-11: now also switch?.1
- net connd-12: now also switch?.2
- net connd-13: now also switch?.1
- net connd-14: now also switch?.2
- net connd-15: now also switch?.1
- net connd-16: now also switch?.2
- net connd-2: now also conn?.3
- net connd-3: now also conn?.1
- net connd-4: now also conn?.2
- net connd-5: now also conn?.3
- net connd-6: now also conn?.1
- net connd-7: now also conn?.2
- net connd-8: now also conn?.3
- net connd-9: now also switch?.1
- net conne-0: now reaches switch?.1
- net conne-0: now also Conn?.1
- net conne-1: now reaches switch?.2
- net conne-1: now also Conn?.2
- net connd-21: now reaches switch?.1
- net connd-21: now also Conn?.22
- net connd-22: now reaches switch?.2
- net connd-22: now also Conn?.23
- net connd-19: now reaches switch?.1
- net connd-19: now also Conn?.20
- net connd-20: now reaches switch?.2
- net connd-20: now also Conn?.21
- net connd-17: now reaches switch?.1
- net connd-17: now also Conn?.18
- net connd-18: now reaches switch?.2
- net connd-18: now also Conn?.19
- net connd-31: now reaches switch?.1
- net connd-31: now also Conn?.32
- net connd-32: now reaches switch?.2
- net connd-32: now also Conn?.33
- net connd-33: now reaches switch?.1
- net connd-33: now also Conn?.34
- net connd-34: now reaches switch?.2
- net connd-34: now also Conn?.35
- net connd-29: now reaches switch?.1
- net connd-29: now also Conn?.30
- net connd-30: now reaches switch?.2
- net connd-30: now also Conn?.31
- net connd-27: now reaches switch?.1
- net connd-27: now also Conn?.28
- net connd-28: now reaches switch?.2
- net connd-28: now also Conn?.29
- net connd-25: now reaches switch?.1
- net connd-25: now also Conn?.26
- net connd-26: now reaches switch?.2
- net connd-26: now also Conn?.27
- net connd-23: now reaches switch?.1
- net connd-23: now also Conn?.24
- net connd-24: now reaches switch?.2
- net connd-24: now also Conn?.25
- net conne-17: now reaches VAC-SEN?.1 (Vcc)
- net conne-17: now also Conn?.18
- net conne-18: now reaches VAC-SEN?.2 (Gnd)
- net conne-18: now also Conn?.19
- net conne-19: now reaches VAC-SEN?.3 (Out)
- net conne-19: now also Conn?.20
- net conne-20: now reaches VAC-SEN?.1 (Vcc)
- net conne-20: now also Conn?.21
- net conne-21: now reaches VAC-SEN?.2 (Gnd)
- net conne-21: now also Conn?.22
- net conne-22: now reaches VAC-SEN?.3 (Out)
- net conne-22: now also Conn?.23
- net conne-23: now reaches VAC-SEN?.1 (Vcc)
- net conne-23: now also Conn?.24
- net conne-24: now reaches VAC-SEN?.2 (Gnd)
- net conne-24: now also Conn?.25
- net conne-25: now reaches VAC-SEN?.3 (Out)
- net conne-25: now also Conn?.26
- net conne-26: now reaches VAC-SEN?.1 (Vcc)
- net conne-26: now also Conn?.27
- net conne-27: now reaches VAC-SEN?.2 (Gnd)
- net conne-27: now also Conn?.28
- net conne-28: now reaches VAC-SEN?.3 (Out)
- net conne-28: now also Conn?.29
- net conne-29: now reaches VAC-SEN?.1 (Vcc)
- net conne-29: now also Conn?.30
- net conne-30: now reaches VAC-SEN?.2 (Gnd)
- net conne-30: now also Conn?.31
- net conne-31: now reaches VAC-SEN?.3 (Out)
- net conne-31: now also Conn?.32
- net conne-14: now reaches VAC-SEN?.1 (Vcc)
- net conne-14: now also Conn?.15
- net conne-15: now reaches VAC-SEN?.2 (Gnd)
- net conne-15: now also Conn?.16
- net conne-16: now reaches VAC-SEN?.3 (Out)
- net conne-16: now also Conn?.17
- net conne-11: now reaches VAC-SEN?.1 (Vcc)
- net conne-11: now also Conn?.12
- net conne-12: now reaches VAC-SEN?.2 (Gnd)
- net conne-12: now also Conn?.13
- net conne-13: now reaches VAC-SEN?.3 (Out)
- net conne-13: now also Conn?.14
- net conne-8: now reaches VAC-SEN?.1 (Vcc)
- net conne-8: now also Conn?.9
- net conne-9: now reaches VAC-SEN?.2 (Gnd)
- net conne-9: now also Conn?.10
- net conne-10: now reaches VAC-SEN?.3 (Out)
- net conne-10: now also Conn?.11
- net conne-5: now reaches VAC-SEN?.1 (Vcc)
- net conne-5: now also Conn?.6
- net conne-6: now reaches VAC-SEN?.2 (Gnd)
- net conne-6: now also Conn?.7
- net conne-7: now reaches VAC-SEN?.3 (Out)
- net conne-7: now also Conn?.8
- net conne-2: now reaches VAC-SEN?.1 (Vcc)
- net conne-2: now also Conn?.3
- net conne-3: now reaches VAC-SEN?.2 (Gnd)
- net conne-3: now also Conn?.4
- net conne-4: now reaches VAC-SEN?.3 (Out)
- net conne-4: now also Conn?.5
- new net connd-35: Conn?.36
- new net connd-36: Conn?.37
- new net conne-32: Conn?.33
- new net conne-33: Conn?.34
- new net conne-34: Conn?.35
- new net conne-35: Conn?.36
- new net conne-36: Conn?.37
- new net connf-0: Conn?.1
- new net connf-1: Conn?.2
- new net connf-10: Conn?.11
- new net connf-11: Conn?.12
- new net connf-12: Conn?.13
- new net connf-13: Conn?.14
- new net connf-14: Conn?.15
- new net connf-15: Conn?.16
- new net connf-16: Conn?.17
- new net connf-17: Conn?.18
- new net connf-18: Conn?.19
- new net connf-19: Conn?.20
- new net connf-2: Conn?.3
- new net connf-20: Conn?.21
- new net connf-21: Conn?.22
- new net connf-22: Conn?.23
- new net connf-23: Conn?.24
- new net connf-24: Conn?.25
- new net connf-25: Conn?.26
- new net connf-26: Conn?.27
- new net connf-27: Conn?.28
- new net connf-28: Conn?.29
- new net connf-29: Conn?.30
- new net connf-3: Conn?.4
- new net connf-30: Conn?.31
- new net connf-31: Conn?.32
- new net connf-32: Conn?.33
- new net connf-33: Conn?.34
- new net connf-34: Conn?.35
- new net connf-35: Conn?.36
- new net connf-36: Conn?.37
- new net connf-4: Conn?.5
- new net connf-5: Conn?.6
- new net connf-6: Conn?.7
- new net connf-7: Conn?.8
- new net connf-8: Conn?.9
- new net connf-9: Conn?.10
Other:
- moved on the sheet: switch?

Commit message: Valve and sensor cables for robot 50.
Parts:
- removed VAC-SEN? (x6): VACUM-RELAY, symbol VACUM-RELAY
- added Conn4: D-SUB-37, symbol D-SUB-37
- gave numbers to parts that had none: 83
Connections:
- net conne-32: now also VAC-SEN2.1 (Vcc)
- net conne-33: now also VAC-SEN2.2 (Gnd)
- net conne-34: now also VAC-SEN2.3 (Out)
- net connf-0: now also VAC-SEN5.1 (Vcc)
- net connf-1: now also VAC-SEN5.2 (Gnd)
- net connf-10: now also VAC-SEN14.2 (Gnd)
- net connf-11: now also VAC-SEN14.3 (Out)
- net connf-12: now also VAC-SEN16.1 (Vcc)
- net connf-13: now also VAC-SEN16.2 (Gnd)
- net connf-14: now also VAC-SEN16.3 (Out)
- net connf-15: now also VAC-SEN18.1 (Vcc)
- net connf-16: now also VAC-SEN18.2 (Gnd)
- net connf-17: now also VAC-SEN18.3 (Out)
- net connf-18: now also VAC-SEN20.1 (Vcc)
- net connf-19: now also VAC-SEN20.2 (Gnd)
- net connf-2: now also VAC-SEN5.3 (Out)
- net connf-20: now also VAC-SEN20.3 (Out)
- net connf-21: now also VAC-SEN22.1 (Vcc)
- net connf-22: now also VAC-SEN22.2 (Gnd)
- net connf-23: now also VAC-SEN22.3 (Out)
- net connf-24: now also VAC-SEN24.1 (Vcc)
- net connf-25: now also VAC-SEN24.2 (Gnd)
- net connf-26: now also VAC-SEN24.3 (Out)
- net connf-27: now also VAC-SEN3.1 (Vcc)
- net connf-28: now also VAC-SEN3.2 (Gnd)
- net connf-29: now also VAC-SEN3.3 (Out)
- net connf-3: now also VAC-SEN8.1 (Vcc)
- net connf-30: now also VAC-SEN6.1 (Vcc)
- net connf-31: now also VAC-SEN6.2 (Gnd)
- net connf-32: now also VAC-SEN6.3 (Out)
- net connf-33: now also VAC-SEN9.1 (Vcc)
- net connf-34: now also VAC-SEN9.2 (Gnd)
- net connf-35: now also VAC-SEN9.3 (Out)
- net connf-36: now also VAC-SEN12.1 (Vcc)
- net connf-4: now also VAC-SEN8.2 (Gnd)
- net connf-5: now also VAC-SEN8.3 (Out)
- net connf-6: now also VAC-SEN11.1 (Vcc)
- net connf-7: now also VAC-SEN11.2 (Gnd)
- net connf-8: now also VAC-SEN11.3 (Out)
- net connf-9: now also VAC-SEN14.1 (Vcc)
- net connf-37: now reaches VAC-SEN12.2 (Gnd)
- net connf-38: now reaches VAC-SEN12.3 (Out)
- new net conng-0: Conn4.1
- new net conng-1: Conn4.2
- new net conng-10: Conn4.11
- new net conng-11: Conn4.12
- new net conng-12: Conn4.13
- new net conng-13: Conn4.14
- new net conng-14: Conn4.15
- new net conng-15: Conn4.16
- new net conng-16: Conn4.17
- new net conng-17: Conn4.18
- new net conng-18: Conn4.19
- new net conng-19: Conn4.20
- new net conng-2: Conn4.3
- new net conng-20: Conn4.21
- new net conng-21: Conn4.22
- new net conng-22: Conn4.23
- new net conng-23: Conn4.24
- new net conng-24: Conn4.25
- new net conng-25: Conn4.26
- new net conng-26: Conn4.27
- new net conng-27: Conn4.28
- new net conng-28: Conn4.29
- new net conng-29: Conn4.30
- new net conng-3: Conn4.4
- new net conng-30: Conn4.31
- new net conng-31: Conn4.32
- new net conng-32: Conn4.33
- new net conng-33: Conn4.34
- new net conng-34: Conn4.35
- new net conng-35: Conn4.36
- new net conng-36: Conn4.37
- new net conng-4: Conn4.5
- new net conng-5: Conn4.6
- new net conng-6: Conn4.7
- new net conng-7: Conn4.8
- new net conng-8: Conn4.9
- new net conng-9: Conn4.10
Other:
- moved on the sheet: VAC-SEN1, VAC-SEN10, VAC-SEN11, VAC-SEN12, VAC-SEN13, VAC-SEN14, VAC-SEN15, VAC-SEN16, VAC-SEN17, VAC-SEN18, VAC-SEN19, VAC-SEN2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

Commit message: Vavle and power cables for new schemas.
Parts:
- removed Conn1, Conn2, Conn3, Conn4, Conn5, Conn6, Conn7: D-SUB-37, symbol D-SUB-37
- removed conn18, conn19, conn20, conn22, conn23, conn24, conn25, conn26, conn27, conn28, conn29, conn30, conn31, conn32, conn33, conn34, conn35, conn36, conn37, conn38, conn39: 122-892P, symbol 122-892P
- removed switch14: DRY-SWITCH, symbol DRY-SWITCH
- added J1, J2, J3, J4, J5, J6: DB37, symbol DB37
- added conn19, conn20: A60, symbol 122-800
- conn1, conn13, conn17, conn5, conn9: value 122-800 -> A60
- conn10, conn11, conn12, conn14, conn15, conn16, conn2, conn3, conn4, conn6, conn7, conn8: value 122-892P -> U73
- conn18: renamed from conn21; value 122-800 -> A60
- switch1: value DRY-SWITCH -> TRP-8
- switch10: renamed from switch11; value DRY-SWITCH -> CST220N2
- switch11: renamed from switch10; value DRY-SWITCH -> CST220N2
- switch12: renamed from switch13; value DRY-SWITCH -> CST220N2
- switch13: renamed from switch12; value DRY-SWITCH -> CST220N2
- switch2: renamed from switch3; value DRY-SWITCH -> CST220N2
- switch3: renamed from switch2; value DRY-SWITCH -> CST220N2
- switch4: renamed from switch5; value DRY-SWITCH -> CST220N2
- switch5: renamed from switch4; value DRY-SWITCH -> CST220N2
- switch6: renamed from switch7; value DRY-SWITCH -> CST220N2
- switch7: renamed from switch6; value DRY-SWITCH -> CST220N2
- switch8: renamed from switch9; value DRY-SWITCH -> CST220N2
- switch9: renamed from switch8; value DRY-SWITCH -> CST220N2
Connections:
- net labels added: A60+1, A60+2, A60+3, A60+4, A60+5, A60+6, A60+7, A60+8, A60-1, A60-2, A60-3, A60-4, A60-5, A60-6, A60-7, A60-8, A60GND1, A60GND2, A60GND3, A60GND4, A60GND5, A60GND6, A60GND7, A60GND8, CABLE1, CABLE2, CABLE3, CABLE4, CABLE5, CABLE6, DS+1, DS+10, DS+11, DS+12, DS+2, DS+3, DS+4, DS+5, DS+6, DS+7, DS+8, DS+9, DS-1, DS-10, DS-11, DS-12, DS-2, DS-3, DS-4, DS-5, DS-6, DS-7, DS-8, DS-9, TRP+, TRP-, U73+1, U73+10, U73+11, U73+12, U73+2, U73+3, U73+4, U73+5, U73+6, U73+7, U73+8, U73+9, U73-1, U73-10, U73-11, U73-12, U73-2, U73-3, U73-4, U73-5, U73-6, U73-7, U73-8, U73-9, VR+1, VR+10, VR+11, VR+12, VR+13, VR+14, VR+15, VR+16, VR+17, VR+18, VR+19, VR+2, VR+20, VR+21, VR+22, VR+23, VR+24, VR+3, VR+4, VR+5, VR+6, VR+7, VR+8, VR+9, VR-1, VR-10, VR-11, VR-12, VR-13, VR-14, VR-15, VR-16, VR-17, VR-18, VR-19, VR-2, VR-20, VR-21, VR-22, VR-23, VR-24, VR-3, VR-4, VR-5, VR-6, VR-7, VR-8, VR-9, VR1, VR10, VR11, VR12, VR13, VR14, VR15, VR16, VR17, VR18, VR19, VR2, VR20, VR21, VR22, VR23, VR24, VR3, VR4, VR5, VR6, VR7, VR8, VR9
- net labels removed: c10[27..29], c11[30..32], c12[33..25], c13[0..2], c14[3..5], c15[6..8], c16[9..11], c17[12..14], c18[15..17], c19[18..20], c1[0..2], c20[21..23], c21[24..26], c22[27..29], c23[30..32], c24[33..35], c25[0..2], c26[3..5], c27[6..8], c28[9..11], c29[12..14], c2[3..5], c30[15..17], c31[18..20], c32[21..23], c33[27..29], c34[27..29], c35[30..32], c36[33..35], c37[0..2], c38[3..5], c39[6..8], c3[6..8], c40[9..10], c41[11..12], c42[13..14], c43[15..16], c44[17..18], c45[19..20], c46[21..22], c47[23..24], c48[25..26], c49[27..28], c4[9..11], c50[29..30], c51[31..32], c52[33.34], c53[0..1], c54[2..4], c55[5..7], c56[8..10], c57[11..13], c58[14..16], c59[17..19], c5[12..14], c60[20..22], c61[23..25], c62[26..28], c63[29..31], c64[32..34], c65[0..2], c66[3..5], c67[6..8], c68[9..11], c69[12..14], c6[15..17], c70[15..17], c71[18..20], c72[21..23], c73[24..26], c74[27..29], c75[30..32], c76[33..35], c77, c7[18..20], c8[21..23], c9[24..26], conna-0, conna-1, conna-10, conna-11, conna-12, conna-13, conna-14, conna-15, conna-16, conna-17, conna-18, conna-19, conna-2, conna-20, conna-21, conna-22, conna-23, conna-24, conna-25, conna-26, conna-27, conna-28, conna-29, conna-3, conna-30, conna-31, conna-32, conna-33, conna-34, conna-35, conna-36, conna-4, conna-5, conna-6, conna-7, conna-8, conna-9, conna[0..36], connb-0, connb-1, connb-10, connb-11, connb-12, connb-13, connb-14, connb-15, connb-16, connb-17, connb-18, connb-19, connb-2, connb-20, connb-21, connb-22, connb-23, connb-24, connb-25, connb-26, connb-27, connb-28, connb-29, connb-3, connb-30, connb-31, connb-32, connb-33, connb-34, connb-35, connb-36, connb-4, connb-5, connb-6, connb-7, connb-8, connb-9, connb[0..36], connc-0, connc-1, connc-10, connc-11, connc-12, connc-13, connc-14, connc-15, connc-16, connc-17, connc-18, connc-19, connc-2, connc-20, connc-21, connc-22, connc-23, connc-24, connc-25, connc-26, connc-27, connc-28, connc-29, connc-3, connc-30, connc-31, connc-32, connc-33, connc-34, connc-35, connc-36, connc-4, connc-5, connc-6, connc-7, connc-8, connc-9, connc[0..36], connd-0, connd-1, connd-10, connd-11, connd-12, connd-13, connd-14, connd-15, connd-16, connd-17, connd-18, connd-19, connd-2, connd-20, connd-21, connd-22, connd-23, connd-24, connd-25, connd-26, connd-27, connd-28, connd-29, connd-3, connd-30, connd-31, connd-32, connd-33, connd-34, connd-35, connd-36, connd-4, connd-5, connd-6, connd-7, connd-8, connd-9, connd[0..36], conne-0, conne-1, conne-10, conne-11, conne-12, conne-13, conne-14, conne-15, conne-16, conne-17, conne-18, conne-19, conne-2, conne-20, conne-21, conne-22, conne-23, conne-24, conne-25, conne-26, conne-27, conne-28, conne-29, conne-3, conne-30, conne-31, conne-32, conne-33, conne-34, conne-35, conne-36, conne-4, conne-5, conne-6, conne-7, conne-8, conne-9, conne[0..36], connf-0, connf-1, connf-10, connf-11, connf-12, connf-13, connf-14, connf-15, connf-16, connf-17, connf-18, connf-19, connf-2, connf-20, connf-21, connf-22, connf-23, connf-24, connf-25, connf-26, connf-27, connf-28, connf-29, connf-3, connf-30, connf-31, connf-32, connf-33, connf-34, connf-35, connf-36, connf-37, connf-38, connf-4, connf-5, connf-6, connf-7, connf-8, connf-9, connf[0..36], conng-0, conng-1, conng-10, conng-11, conng-12, conng-13, conng-14, conng-15, conng-16, conng-17, conng-18, conng-19, conng-2, conng-20, conng-21, conng-22, conng-23, conng-24, conng-25, conng-26, conng-27, conng-28, conng-29, conng-3, conng-30, conng-31, conng-32, conng-33, conng-34, conng-35, conng-36, conng-4, conng-5, conng-6, conng-7, conng-8, conng-9, conng[0..36]
- wire segments 476 -> 380
Other:
- note added: "Magnetic position sensor CST220N2 - 12"
- note added: "Memory valves A60 - 8"
- note added: "Model "50" IO table"
- note added: "Pressure relay TRP8 - 1"
- note added: "Regular valves U73 - 12"
- note added: "Vacum relays SWM-VD6-T6 - 24"
- moved on the sheet: VAC-SEN1, VAC-SEN10, VAC-SEN11, VAC-SEN12, VAC-SEN13, VAC-SEN14, VAC-SEN15, VAC-SEN16, VAC-SEN17, VAC-SEN18, VAC-SEN19, VAC-SEN2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
