File: schema/moto_ctrl/moto_ctrl.sch (KiCad schematic (older format))
At the start: 98 parts, among them J1 DB9, J2 DB37, K1 i2c-1, P1 CONN_2, P2 SWD-IAP, U1 NCP3063, U2 MINI-USB-B, X1 8MHz

Commit message: Added analog part of revolution motor control.
Parts:
- added C18, C19, C20: 10u, symbol C
- added P2: power-1, symbol CONN_12
- added P3: power-2, symbol CONN_12
- renumbered C10 to C1, C15 to C10, C16 to C11, C17 to C12, C2 to C13, C3 to C14, C9 to C15, C7 to C16, C8 to C17, C11 to C2, C18 to C21, C19 to C22, C20 to C23, C21 to C24, C12 to C3, C13 to C4, C1 to C5, C4 to C6, C5 to C7, C6 to C8, C14 to C9, D3 to D1, D1 to D2, D2 to D3, J2 to J1, J1 to J2, P2 to P4, R2 to R1, R26 to R10, R33 to R11, R42 to R12, R52 to R13, R28 to R14, R37 to R15, R46 to R16, R54 to R17, R25 to R18, R34 to R19, R5 to R2, R35 to R20, R43 to R21, R44 to R22, R50 to R23, R51 to R24, R59 to R25, R60 to R26, R31 to R27, R40 to R28, R61 to R29, R7 to R3, R57 to R30, R32 to R31, R41 to R32, R49 to R33, R58 to R34, R29 to R35, R38 to R36, R47 to R37, R55 to R38, R1 to R39, R21 to R4, R6 to R40, R30 to R41, R39 to R42, R48 to R43, R56 to R44, R24 to R45, R22 to R46, R23 to R47, R4 to R48, R8 to R49, R27 to R5, R11 to R50, R18 to R51, R19 to R52, R20 to R53, R12 to R54, R16 to R55, R17 to R56, R13 to R57, R62 to R58, R63 to R59, R36 to R6, R14 to R60, R9 to R61, R10 to R62, R3 to R63, R45 to R7, R53 to R8, R15 to R9
Connections:
- net labels added: +5V
- wire segments 339 -> 401

Commit message: Added analog outputs for escon 50/5 controls, rs-485 inputs for encoder signals recognition and DB-9 sockets for encoder inputs.
Connections:
- net labels added: an-out1, an-out2, an-out3, an-out4
- wire segments 401 -> 411
- no-connect marks 12 -> 7

Commit message: Schema edited. Have to leave just tow manipulator controls on one board. So it will be two boards for total control. Painted PCB edge with placment holes identical to previous valve_2 PCB.
Parts:
- removed C11, C12: 100n, symbol C
- removed C20: 10u, symbol C
- removed R12, R13, R29, R30, R33, R34, R37, R38, R43, R44: 100, symbol R
- removed R16, R17, R23, R24, R25, R26: 10k, symbol R
- removed R7: 81k, symbol R
- removed R8: 80k, symbol R
- added C11: 54u, symbol CP1
- added K?: i2c-1, symbol CONN_3
- added P5, P6: CONN_2, symbol CONN_2
Connections:
- net labels removed: an-out3, an-out4, dr-gnd-3, dr-gnd-4, dr-i-31, dr-i-32, dr-i-41, dr-i-42, dr-io-31, dr-io-32, dr-io-41, dr-io-42, i-3-1, i-3-2, i-4-1, i-4-2, io-3-1, io-3-2, io-4-1, io-4-2, sen-3, sen-4, sen-gnd-3, sen-gnd-4, sen-vdd-3, sen-vdd-4, sensor-3, sensor-4
- wire segments 411 -> 338
- no-connect marks 7 -> 36
Other:
- note added: "Driver power socket (output)"
- note added: "High power input"
- moved on the sheet: J1

Commit message: Started routing. At the moment don't know where I should put clemmas power. Probably replace D-SUB-9 with them.
Parts:
- removed P1: CONN_2, symbol CONN_2
- added P1: SETUP, symbol CONN_8
- added R12, R7, R8: 10k, symbol R
- P5: value CONN_2 -> PWR-IN
- P6: value CONN_2 -> PWR-OUT
- gave numbers to parts that had none: 1
Connections:
- net labels added: addr0, addr1, addr2
- wire segments 338 -> 357
- no-connect marks 36 -> 33

Commit message: Placing elements.
Parts:
- removed J2: DB9, symbol DB9
Connections:
- net labels removed: 24v, gnd
- wire segments 357 -> 348
- no-connect marks 33 -> 35
