File: schema/moto_ctrl/moto_ctrl.sch (KiCad schematic (older format))
At the start: 88 parts, among them J1 DB37, K1 i2c-1, K2 i2c-1, P1 SETUP, P2 power-1, P3 power-2, P4 SWD-IAP, P5 PWR-IN, P6 PWR-OUT, U1 NCP3063, U2 MINI-USB-B, X1 8MHz

Commit message: Made switchable USB.
Parts:
- added R13: 1k5, symbol R
- added R16: 15k, symbol R
Connections:
- net labels added: usb-en
- wire segments 348 -> 356
Other:
- note added: "Here it should be either MCU pin USB ctrl \nor just direct pullup. NOT both of them!!!"
- moved on the sheet: P4, R54, R55, R56, R57, R60
